Commit message: lrmate200ic: update urdfs based on DH data. For ros-industrial/fanuc#54 and ros-industrial/fanuc#63.

File: fanuc_lrmate200ic_support/urdf/lrmate200ic.urdf (robot description, URDF)
Before this commit: robot fanuc_lrmate200ic, 8 links, 7 joints
Joints:
- joint joint_1: origin xyz=0 0 0.33 rpy=0 0 0 -> xyz=0 0 0.330 rpy=0 0 0
- joint joint_3: origin xyz=0 0 0.3 rpy=0 0 0 -> xyz=0 0 0.300 rpy=0 0 0
- joint joint_4: origin xyz=0.32 0 0.075 rpy=0 0 0 -> xyz=0 0 0.075 rpy=0 0 0
- joint joint_5: origin xyz=0 0 0 rpy=0 0 0 -> xyz=0.320 0 0 rpy=0 0 0
- joint joint_6: axis 0 0 -1 -> -1 0 0; origin xyz=0.08 0 0 rpy=3.1416 -1.5708 0 -> xyz=0.080 0 0 rpy=0 0 0
- joint joint_6-tool0: origin xyz=0 0 0 rpy=0 0 0 -> xyz=0 0 0 rpy=3.1415926535 -1.570796327 0

File: fanuc_lrmate200ic_support/urdf/lrmate200ic5h.urdf (robot description, URDF)
Before this commit: robot fanuc_lrmate200ic5h, 7 links, 6 joints
Joints:
- joint joint_1: origin xyz=0 0 0.33 rpy=0 0 0 -> xyz=0 0 0.330 rpy=0 0 0
- joint joint_3: origin xyz=0 0 0.3 rpy=0 0 0 -> xyz=0 0 0.300 rpy=0 0 0
- joint joint_4: origin xyz=0.32 0 0.075 rpy=0 0 0 -> xyz=0.320 0 0.075 rpy=0 0 0
- joint joint_5: axis 0 0 -1 -> -1 0 0; origin xyz=0.08 0 0 rpy=1.5708 -1.4902 1.5708 -> xyz=0.080 0 0 rpy=0 0 0
- joint joint_5-tool0: origin xyz=0 0 0 rpy=0 0 0 -> xyz=0 0 0 rpy=3.1415926535 -1.570796327 0

File: fanuc_lrmate200ic_support/urdf/lrmate200ic5h_macro.xacro (robot description, xacro)
@@ -2,4 +2,5 @@
 <robot xmlns:xacro="http://ros.org/wiki/xacro">
 	<xacro:include filename="$(find fanuc_assets)/urdf/common_materials.xacro"/>
+	<xacro:include filename="$(find fanuc_assets)/urdf/common_constants.xacro"/>
 	<xacro:macro name="fanuc_lrmate200ic5h" params="prefix">
 		<link name="${prefix}base_link">
@@ -80,5 +81,5 @@
 		<link name="${prefix}link_5">
 			<visual>
-				<origin xyz="0 0 0" rpy="0 0 0" />
+				<origin xyz="0 0 0" rpy="0 0 0"/>
 				<geometry>
 					<mesh filename="package://fanuc_lrmate200ic_support/meshes/lrmate200ic/visual/link_6.stl" />
@@ -87,5 +88,5 @@
 			</visual>
 			<collision>
-				<origin xyz="0 0 0" rpy="0 0 0" />
+				<origin xyz="0 0 0" rpy="0 0 0"/>
 				<geometry>
 					<mesh filename="package://fanuc_lrmate200ic_support/meshes/lrmate200ic/collision/link_6.stl" />
@@ -95,5 +96,5 @@
 		<link name="${prefix}tool0" />
 		<joint name="${prefix}joint_1" type="revolute">
-			<origin xyz="0 0 0.33" rpy="0 0 0" />
+			<origin xyz="0 0 0.330" rpy="0 0 0" />
 			<parent link="${prefix}base_link" />
 			<child link="${prefix}link_1" />
@@ -109,5 +110,5 @@
 		</joint>
 		<joint name="${prefix}joint_3" type="revolute">
-			<origin xyz="0 0 0.3" rpy="0 0 0" />
+			<origin xyz="0 0 0.300" rpy="0 0 0" />
 			<parent link="${prefix}link_2" />
 			<child link="${prefix}link_3" />
@@ -116,5 +117,5 @@
 		</joint>
 		<joint name="${prefix}joint_4" type="revolute">
-			<origin xyz="0.32 0 0.075" rpy="0 0 0" />
+			<origin xyz="0.320 0 0.075" rpy="0 0 0" />
 			<parent link="${prefix}link_3" />
 			<child link="${prefix}link_4" />
@@ -123,14 +124,14 @@
 		</joint>
 		<joint name="${prefix}joint_5" type="revolute">
-			<origin xyz="0.08 0 0" rpy="1.5708 -1.4902 1.5708" />
+			<origin xyz="0.080 0 0" rpy="0 0 0" />
 			<parent link="${prefix}link_4" />
 			<child link="${prefix}link_5" />
-			<axis xyz="0 0 -1" />
+			<axis xyz="-1 0 0" />
 			<limit effort="0" lower="-6.285" upper="6.285" velocity="12.5664" />
 		</joint>
 		<joint name="${prefix}joint_5-tool0" type="fixed">
+			<origin xyz="0 0 0" rpy="${m_pi} ${-m_pi_2} 0" />
 			<parent link="${prefix}link_5" />
 			<child link="${prefix}tool0" />
-			<origin xyz="0 0 0" rpy="0 0 0" />
 		</joint>
 	</xacro:macro>

File: fanuc_lrmate200ic_support/urdf/lrmate200ic_macro.xacro (robot description, xacro)
@@ -2,4 +2,5 @@
 <robot xmlns:xacro="http://ros.org/wiki/xacro">
 	<xacro:include filename="$(find fanuc_assets)/urdf/common_materials.xacro"/>
+	<xacro:include filename="$(find fanuc_assets)/urdf/common_constants.xacro"/>
 	<xacro:macro name="fanuc_lrmate200ic" params="prefix">
 		<link name="${prefix}base_link">
@@ -110,5 +111,5 @@
 		<link name="${prefix}tool0" />
 		<joint name="${prefix}joint_1" type="revolute">
-			<origin xyz="0 0 0.33" rpy="0 0 0" />
+			<origin xyz="0 0 0.330" rpy="0 0 0" />
 			<parent link="${prefix}base_link" />
 			<child link="${prefix}link_1" />
@@ -124,5 +125,5 @@
 		</joint>
 		<joint name="${prefix}joint_3" type="revolute">
-			<origin xyz="0 0 0.3" rpy="0 0 0" />
+			<origin xyz="0 0 0.300" rpy="0 0 0" />
 			<parent link="${prefix}link_2" />
 			<child link="${prefix}link_3" />
@@ -131,5 +132,5 @@
 		</joint>
 		<joint name="${prefix}joint_4" type="revolute">
-			<origin xyz="0.32 0 0.075" rpy="0 0 0"/>
+			<origin xyz="0 0 0.075" rpy="0 0 0"/>
 			<parent link="${prefix}link_3"/>
 			<child link="${prefix}link_4"/>
@@ -138,5 +139,5 @@
 		</joint>
 		<joint name="${prefix}joint_5" type="revolute">
-			<origin xyz="0 0 0" rpy="0 0 0"/>
+			<origin xyz="0.320 0 0" rpy="0 0 0"/>
 			<parent link="${prefix}link_4"/>
 			<child link="${prefix}link_5"/>
@@ -145,14 +146,14 @@
 		</joint>
 		<joint name="${prefix}joint_6" type="revolute">
-			<origin xyz="0.08 0 0" rpy="3.1416 -1.5708 0"/>
+			<origin xyz="0.080 0 0" rpy="0 0 0"/>
 			<parent link="${prefix}link_5"/>
 			<child link="${prefix}link_6"/>
-			<axis xyz="0 0 -1"/>
+			<axis xyz="-1 0 0"/>
 			<limit effort="0" lower="-6.2832" upper="6.2832" velocity="12.5664" />
 		</joint>
 		<joint name="${prefix}joint_6-tool0" type="fixed">
+			<origin xyz="0 0 0" rpy="${m_pi} ${-m_pi_2} 0" />
 			<parent link="${prefix}link_6" />
 			<child link="${prefix}tool0" />
-			<origin xyz="0 0 0" rpy="0 0 0" />
 		</joint>
 	</xacro:macro>

Commit message: lrmate200ic: add 'base' link (transform to World Coordinates). For ros-industrial/fanuc#101.

File: fanuc_lrmate200ic_support/urdf/lrmate200ic.urdf (robot description, URDF)
Before this commit: robot fanuc_lrmate200ic, 8 links, 7 joints
Links:
- added link base
Joints:
- added joint base_link-base: type fixed, parent base_link, child base, origin xyz=0 0 0.330 rpy=0 0 0

File: fanuc_lrmate200ic_support/urdf/lrmate200ic5h.urdf (robot description, URDF)
Before this commit: robot fanuc_lrmate200ic5h, 7 links, 6 joints
Links:
- added link base
Joints:
- added joint base_link-base: type fixed, parent base_link, child base, origin xyz=0 0 0.330 rpy=0 0 0

File: fanuc_lrmate200ic_support/urdf/lrmate200ic5h_macro.xacro (robot description, xacro)
@@ -135,4 +135,11 @@
 			<child link="${prefix}tool0" />
 		</joint>
+		<!-- ROS base_link to Fanuc World Coordinates transform -->
+		<link name="${prefix}base" />
+		<joint name="${prefix}base_link-base" type="fixed">
+			<origin xyz="0 0 0.330" rpy="0 0 0"/>
+			<parent link="${prefix}base_link"/>
+			<child link="${prefix}base"/>
+		</joint>
 	</xacro:macro>
 </robot>

File: fanuc_lrmate200ic_support/urdf/lrmate200ic_macro.xacro (robot description, xacro)
@@ -157,4 +157,11 @@
 			<child link="${prefix}tool0" />
 		</joint>
+		<!-- ROS base_link to Fanuc World Coordinates transform -->
+		<link name="${prefix}base" />
+		<joint name="${prefix}base_link-base" type="fixed">
+			<origin xyz="0 0 0.330" rpy="0 0 0"/>
+			<parent link="${prefix}base_link"/>
+			<child link="${prefix}base"/>
+		</joint>
 	</xacro:macro>
 </robot>
