Commit message: lrmate200ic5f: fix link_4 length.
Misread spec sheet. Link was 0.5mm too short. This caused the Cartesian pose
reported for tool0 to be incorrect.

File: fanuc_lrmate200ic_support/urdf/lrmate200ic5f.urdf (robot description, URDF)
Before this commit: robot fanuc_lrmate200ic5f, 8 links, 7 joints
Joints:
- joint joint_4: origin xyz=0.327 0 0.075 rpy=0 0 0 -> xyz=0.3275 0 0.075 rpy=0 0 0

File: fanuc_lrmate200ic_support/urdf/lrmate200ic5f_macro.xacro (robot description, xacro)
@@ -117,5 +117,5 @@
     </joint>
     <joint name="${prefix}joint_4" type="revolute">
-      <origin xyz="0.327 0 0.075" rpy="0 0 0" />
+      <origin xyz="0.3275 0 0.075" rpy="0 0 0" />
       <parent link="${prefix}link_3" />
       <child link="${prefix}link_4" />
