Commit message: m20ia: update urdfs based on DH data. For ros-industrial/fanuc#54 and ros-industrial/fanuc#63.

File: fanuc_m20ia_support/urdf/m20ia.urdf (robot description, URDF)
Before this commit: robot fanuc_m20ia, 8 links, 7 joints
Joints:
- joint joint_2: origin xyz=0.15 0 0 rpy=0 0 0 -> xyz=0.150 0 0 rpy=0 0 0
- joint joint_3: origin xyz=0 0 0.79 rpy=0 0 0 -> xyz=0 0 0.790 rpy=0 0 0
- joint joint_4: origin xyz=0.22209 0 0.25 rpy=0 0 0 -> xyz=0 0 0.250 rpy=0 0 0
- joint joint_5: origin xyz=0.61291 0 0 rpy=0 0 0 -> xyz=0.835 0 0 rpy=0 0 0
- joint joint_6: origin xyz=0.1 0 0 rpy=0 0 0 -> xyz=0.100 0 0 rpy=0 0 0
- joint joint_6-tool0: origin xyz=0 0 0 rpy=0 0 0 -> xyz=0 0 0 rpy=3.1415926535 -1.570796327 0

File: fanuc_m20ia_support/urdf/m20ia10l.urdf (robot description, URDF)
Before this commit: robot fanuc_m20ia10l, 8 links, 7 joints
Joints:
- joint joint_2: origin xyz=0.15 0 0 rpy=0 0 0 -> xyz=0.150 0 0 rpy=0 0 0
- joint joint_3: origin xyz=0 0 0.79 rpy=0 0 0 -> xyz=0 0 0.790 rpy=0 0 0
- joint joint_4: origin xyz=0 0 0.25 rpy=0 0 0 -> xyz=0 0 0.250 rpy=0 0 0
- joint joint_5: origin xyz=1.04 -0.053 0 rpy=0 0 0 -> xyz=1.040 0 0 rpy=0 0 0
- joint joint_6: origin xyz=0.1 0.053 0 rpy=0 0 0 -> xyz=0.100 0 0 rpy=0 0 0
- joint joint_6-tool0: origin xyz=0 0 0 rpy=0 0 0 -> xyz=0 0 0 rpy=3.1415926535 -1.570796327 0

File: fanuc_m20ia_support/urdf/m20ia10l_macro.xacro (robot description, xacro)
@@ -2,4 +2,5 @@
 <robot xmlns:xacro="http://ros.org/wiki/xacro">
 	<xacro:include filename="$(find fanuc_resources)/urdf/common_materials.xacro"/>
+	<xacro:include filename="$(find fanuc_resources)/urdf/common_constants.xacro"/>
 	<xacro:macro name="fanuc_m20ia10l" params="prefix">
 		<!-- links -->
@@ -119,5 +120,5 @@
 		</joint>
 		<joint name="${prefix}joint_2" type="revolute">
-			<origin xyz="0.15 0 0" rpy="0 0 0"/>
+			<origin xyz="0.150 0 0" rpy="0 0 0"/>
 			<parent link="${prefix}link_1"/>
 			<child link="${prefix}link_2"/>
@@ -126,5 +127,5 @@
 		</joint>
 		<joint name="${prefix}joint_3" type="revolute">
-			<origin xyz="0 0 0.79" rpy="0 0 0"/>
+			<origin xyz="0 0 0.790" rpy="0 0 0"/>
 			<parent link="${prefix}link_2"/>
 			<child link="${prefix}link_3"/>
@@ -133,5 +134,5 @@
 		</joint>
 		<joint name="${prefix}joint_4" type="revolute">
-			<origin xyz="0 0 0.25" rpy="0 0 0"/>
+			<origin xyz="0 0 0.250" rpy="0 0 0"/>
 			<parent link="${prefix}link_3"/>
 			<child link="${prefix}link_4"/>
@@ -140,5 +141,5 @@
 		</joint>
 		<joint name="${prefix}joint_5" type="revolute">
-			<origin xyz="1.04 -0.053 0" rpy="0 0 0"/>
+			<origin xyz="1.040 0 0" rpy="0 0 0"/>
 			<parent link="${prefix}link_4"/>
 			<child link="${prefix}link_5"/>
@@ -147,5 +148,5 @@
 		</joint>
 		<joint name="${prefix}joint_6" type="revolute">
-			<origin xyz="0.1 0.053 0" rpy="0 0 0"/>
+			<origin xyz="0.100 0 0" rpy="0 0 0"/>
 			<parent link="${prefix}link_5"/>
 			<child link="${prefix}link_6"/>
@@ -154,7 +155,7 @@
 		</joint>
 		<joint name="${prefix}joint_6-tool0" type="fixed">
+			<origin xyz="0 0 0" rpy="${m_pi} ${-m_pi_2} 0" />
 			<parent link="${prefix}link_6"/>
 			<child link="${prefix}tool0"/>
-			<origin xyz="0 0 0" rpy="0 0 0"/>
 		</joint>
 	</xacro:macro>

File: fanuc_m20ia_support/urdf/m20ia_macro.xacro (robot description, xacro)
@@ -2,4 +2,5 @@
 <robot xmlns:xacro="http://ros.org/wiki/xacro">
 	<xacro:include filename="$(find fanuc_resources)/urdf/common_materials.xacro"/>
+	<xacro:include filename="$(find fanuc_resources)/urdf/common_constants.xacro"/>
 	<xacro:macro name="fanuc_m20ia" params="prefix">
 		<!-- links -->
@@ -119,5 +120,5 @@
 		</joint>
 		<joint name="${prefix}joint_2" type="revolute">
-			<origin xyz="0.15 0 0" rpy="0 0 0"/>
+			<origin xyz="0.150 0 0" rpy="0 0 0"/>
 			<parent link="${prefix}link_1"/>
 			<child link="${prefix}link_2"/>
@@ -126,5 +127,5 @@
 		</joint>
 		<joint name="${prefix}joint_3" type="revolute">
-			<origin xyz="0 0 0.79" rpy="0 0 0"/>
+			<origin xyz="0 0 0.790" rpy="0 0 0"/>
 			<parent link="${prefix}link_2"/>
 			<child link="${prefix}link_3"/>
@@ -133,5 +134,5 @@
 		</joint>
 		<joint name="${prefix}joint_4" type="revolute">
-			<origin xyz="0.22209 0 0.25" rpy="0 0 0"/>
+			<origin xyz="0 0 0.250" rpy="0 0 0"/>
 			<parent link="${prefix}link_3"/>
 			<child link="${prefix}link_4"/>
@@ -140,5 +141,5 @@
 		</joint>
 		<joint name="${prefix}joint_5" type="revolute">
-			<origin xyz="0.61291 0 0" rpy="0 0 0"/>
+			<origin xyz="0.835 0 0" rpy="0 0 0"/>
 			<parent link="${prefix}link_4"/>
 			<child link="${prefix}link_5"/>
@@ -147,5 +148,5 @@
 		</joint>
 		<joint name="${prefix}joint_6" type="revolute">
-			<origin xyz="0.1 0 0" rpy="0 0 0"/>
+			<origin xyz="0.100 0 0" rpy="0 0 0"/>
 			<parent link="${prefix}link_5"/>
 			<child link="${prefix}link_6"/>
@@ -154,7 +155,7 @@
 		</joint>
 		<joint name="${prefix}joint_6-tool0" type="fixed">
+			<origin xyz="0 0 0" rpy="${m_pi} ${-m_pi_2} 0" />
 			<parent link="${prefix}link_6"/>
 			<child link="${prefix}tool0"/>
-			<origin xyz="0 0 0" rpy="0 0 0"/>
 		</joint>
 	</xacro:macro>

Commit message: m20ia: add 'base' link (transform to World Coordinates). For ros-industrial/fanuc#101.

File: fanuc_m20ia_support/urdf/m20ia.urdf (robot description, URDF)
Before this commit: robot fanuc_m20ia, 8 links, 7 joints
Links:
- added link base
Joints:
- added joint base_link-base: type fixed, parent base_link, child base, origin xyz=0 0 0.525 rpy=0 0 0

File: fanuc_m20ia_support/urdf/m20ia10l.urdf (robot description, URDF)
Before this commit: robot fanuc_m20ia10l, 8 links, 7 joints
Links:
- added link base
Joints:
- added joint base_link-base: type fixed, parent base_link, child base, origin xyz=0 0 0.525 rpy=0 0 0

File: fanuc_m20ia_support/urdf/m20ia10l_macro.xacro (robot description, xacro)
@@ -159,4 +159,11 @@
 			<child link="${prefix}tool0"/>
 		</joint>
+		<!-- ROS base_link to Fanuc World Coordinates transform -->
+		<link name="${prefix}base" />
+		<joint name="${prefix}base_link-base" type="fixed">
+			<origin xyz="0 0 0.525" rpy="0 0 0"/>
+			<parent link="${prefix}base_link"/>
+			<child link="${prefix}base"/>
+		</joint>
 	</xacro:macro>
 </robot>

File: fanuc_m20ia_support/urdf/m20ia_macro.xacro (robot description, xacro)
@@ -159,4 +159,11 @@
 			<child link="${prefix}tool0"/>
 		</joint>
+		<!-- ROS base_link to Fanuc World Coordinates transform -->
+		<link name="${prefix}base" />
+		<joint name="${prefix}base_link-base" type="fixed">
+			<origin xyz="0 0 0.525" rpy="0 0 0"/>
+			<parent link="${prefix}base_link"/>
+			<child link="${prefix}base"/>
+		</joint>
 	</xacro:macro>
 </robot>
