Commit message: Removed myself as a maintainer

File: fanuc_cr7ia_support/urdf/cr7ial_macro.xacro (robot description, xacro)
@@ -1,4 +1,5 @@
 <?xml version="1.0" ?>
 <robot xmlns:xacro="http://ros.org/wiki/xacro">
+  <xacro:property name="pi" value="3.1415926535897931" />
   <xacro:include filename="$(find fanuc_resources)/urdf/common_materials.xacro"/>
   <xacro:macro name="fanuc_cr7ial" params="prefix">

Commit message: Updated joint limits and the manual used to get them

File: fanuc_cr7ia_support/urdf/cr7ial_macro.xacro (robot description, xacro)
@@ -1,5 +1,4 @@
 <?xml version="1.0" ?>
 <robot xmlns:xacro="http://ros.org/wiki/xacro">
-  <xacro:property name="pi" value="3.1415926535897931" />
   <xacro:include filename="$(find fanuc_resources)/urdf/common_materials.xacro"/>
   <xacro:macro name="fanuc_cr7ial" params="prefix">
@@ -123,5 +122,5 @@
       <child link="${prefix}link_2" />
       <axis xyz="0 1 0" />
-      <limit effort="0" lower="-1.5708" upper="2.4435" velocity="4.7124" />
+      <limit effort="0" lower="-1.15192" upper="1.74533" velocity="4.7124" />
     </joint>
     <joint name="${prefix}joint_3" type="revolute">
@@ -130,5 +129,5 @@
       <child link="${prefix}link_3" />
       <axis xyz="0 -1 0" />
-      <limit effort="0" lower="-2.5831" upper="4.0143" velocity="4.7124" />
+      <limit effort="0" lower="-0.802851" upper="3.10669" velocity="4.7124" />
     </joint>
     <joint name="${prefix}joint_4" type="revolute">

Commit message: cr7ia: set /L limits based on sysvars.

File: fanuc_cr7ia_support/urdf/cr7ial_macro.xacro (robot description, xacro)
@@ -115,5 +115,5 @@
       <child link="${prefix}link_1" />
       <axis xyz="0 0 1" />
-      <limit effort="0" lower="-2.9671" upper="2.9671" velocity="4.7124" />
+      <limit effort="0" lower="-2.9671" upper="2.9671" velocity="6.4577" />
     </joint>
     <joint name="${prefix}joint_2" type="revolute">
@@ -122,5 +122,5 @@
       <child link="${prefix}link_2" />
       <axis xyz="0 1 0" />
-      <limit effort="0" lower="-1.15192" upper="1.74533" velocity="4.7124" />
+      <limit effort="0" lower="-1.15192" upper="1.74533" velocity="5.4105" />
     </joint>
     <joint name="${prefix}joint_3" type="revolute">
@@ -129,5 +129,5 @@
       <child link="${prefix}link_3" />
       <axis xyz="0 -1 0" />
-      <limit effort="0" lower="-0.802851" upper="3.10669" velocity="4.7124" />
+      <limit effort="0" lower="-0.802851" upper="3.10669" velocity="7.1558" />
     </joint>
     <joint name="${prefix}joint_4" type="revolute">
@@ -136,5 +136,5 @@
       <child link="${prefix}link_4"/>
       <axis xyz="-1 0 0"/>
-      <limit effort="0" lower="-3.3161" upper="3.3161" velocity="7.8540" />
+      <limit effort="0" lower="-3.3161" upper="3.3161" velocity="9.5993" />
     </joint>
     <joint name="${prefix}joint_5" type="revolute">
@@ -143,5 +143,5 @@
       <child link="${prefix}link_5"/>
       <axis xyz="0 -1 0"/>
-      <limit effort="0" lower="-2.0944" upper="2.0944" velocity="7.8540" />
+      <limit effort="0" lower="-2.0944" upper="2.0944" velocity="9.5120" />
     </joint>
     <joint name="${prefix}joint_6" type="revolute">
@@ -150,5 +150,5 @@
       <child link="${prefix}link_6"/>
       <axis xyz="-1 0 0"/>
-      <limit effort="0" lower="-6.2832" upper="6.2832" velocity="12.5664" />
+      <limit effort="0" lower="-6.2832" upper="6.2832" velocity="17.4532" />
     </joint>
     <!-- ROS-Industrial 'base' frame: base_link to Fanuc World Coordinates transform -->

Commit message: Reduced meshes so cr7ia is the base model and cr7ial extends only the different meshes

File: fanuc_cr7ia_support/urdf/cr7ial_macro.xacro (robot description, xacro)
@@ -8,5 +8,5 @@
         <origin xyz="0 0 0" rpy="0 0 0"/>
         <geometry>
-          <mesh filename="package://fanuc_cr7ia_support/meshes/cr7ial/visual/base_link.stl"/>
+          <mesh filename="package://fanuc_cr7ia_support/meshes/cr7ia/visual/base_link.stl"/>
         </geometry>
         <xacro:material_fanuc_gray24 />
@@ -15,5 +15,5 @@
         <origin xyz="0 0 0" rpy="0 0 0"/>
         <geometry>
-          <mesh filename="package://fanuc_cr7ia_support/meshes/cr7ial/collision/base_link.stl"/>
+          <mesh filename="package://fanuc_cr7ia_support/meshes/cr7ia/collision/base_link.stl"/>
         </geometry>
       </collision>
@@ -23,5 +23,5 @@
         <origin xyz="0 0 0" rpy="0 0 0"/>
         <geometry>
-          <mesh filename="package://fanuc_cr7ia_support/meshes/cr7ial/visual/link_1.stl"/>
+          <mesh filename="package://fanuc_cr7ia_support/meshes/cr7ia/visual/link_1.stl"/>
         </geometry>
         <xacro:material_fanuc_green />
@@ -30,5 +30,5 @@
         <origin xyz="0 0 0" rpy="0 0 0"/>
         <geometry>
-          <mesh filename="package://fanuc_cr7ia_support/meshes/cr7ial/collision/link_1.stl"/>
+          <mesh filename="package://fanuc_cr7ia_support/meshes/cr7ia/collision/link_1.stl"/>
         </geometry>
       </collision>
@@ -53,5 +53,5 @@
         <origin xyz="0 0 0" rpy="0 0 0"/>
         <geometry>
-          <mesh filename="package://fanuc_cr7ia_support/meshes/cr7ial/visual/link_3.stl"/>
+          <mesh filename="package://fanuc_cr7ia_support/meshes/cr7ia/visual/link_3.stl"/>
         </geometry>
         <xacro:material_fanuc_green />
@@ -60,5 +60,5 @@
         <origin xyz="0 0 0" rpy="0 0 0"/>
         <geometry>
-          <mesh filename="package://fanuc_cr7ia_support/meshes/cr7ial/collision/link_3.stl"/>
+          <mesh filename="package://fanuc_cr7ia_support/meshes/cr7ia/collision/link_3.stl"/>
         </geometry>
       </collision>
@@ -83,5 +83,5 @@
         <origin xyz="0 0 0" rpy="0 0 0"/>
         <geometry>
-          <mesh filename="package://fanuc_cr7ia_support/meshes/cr7ial/visual/link_5.stl"/>
+          <mesh filename="package://fanuc_cr7ia_support/meshes/cr7ia/visual/link_5.stl"/>
         </geometry>
         <xacro:material_fanuc_green />
@@ -90,5 +90,5 @@
         <origin xyz="0 0 0" rpy="0 0 0"/>
         <geometry>
-          <mesh filename="package://fanuc_cr7ia_support/meshes/cr7ial/collision/link_5.stl"/>
+          <mesh filename="package://fanuc_cr7ia_support/meshes/cr7ia/collision/link_5.stl"/>
         </geometry>
       </collision>
@@ -98,5 +98,5 @@
         <origin xyz="0 0 0" rpy="0 0 0"/>
         <geometry>
-          <mesh filename="package://fanuc_cr7ia_support/meshes/cr7ial/visual/link_6.stl"/>
+          <mesh filename="package://fanuc_cr7ia_support/meshes/cr7ia/visual/link_6.stl"/>
         </geometry>
         <xacro:material_fanuc_gray24 />
@@ -105,5 +105,5 @@
         <origin xyz="0 0 0" rpy="0 0 0"/>
         <geometry>
-          <mesh filename="package://fanuc_cr7ia_support/meshes/cr7ial/collision/link_6.stl"/>
+          <mesh filename="package://fanuc_cr7ia_support/meshes/cr7ia/collision/link_6.stl"/>
         </geometry>
       </collision>
