Commit message: Use as many links as possible from the M-710iC50

File: fanuc_m710ic_support/urdf/m710ic45m_macro.xacro (robot description, xacro)
@@ -2,4 +2,5 @@
 <robot xmlns:xacro="http://wiki.ros.org/xacro">
   <xacro:include filename="$(find fanuc_resources)/urdf/common_materials.xacro"/>
+  <!-- Only link 2 and 4 differ from a M-710iC50 so we re-use them -->
   <xacro:macro name="fanuc_m710ic45m" params="prefix">
     <!-- links: main serial chain -->
@@ -8,5 +9,5 @@
         <origin xyz="0 0 0" rpy="0 0 0"/>
         <geometry>
-          <mesh filename="package://fanuc_m710ic_support/meshes/m710ic45m/visual/base_link.stl"/>
+          <mesh filename="package://fanuc_m710ic_support/meshes/m710ic50/visual/base_link.stl"/>
         </geometry>
         <xacro:material_fanuc_black />
@@ -15,5 +16,5 @@
         <origin xyz="0 0 0" rpy="0 0 0"/>
         <geometry>
-          <mesh filename="package://fanuc_m710ic_support/meshes/m710ic45m/collision/base_link.stl"/>
+          <mesh filename="package://fanuc_m710ic_support/meshes/m710ic50/collision/base_link.stl"/>
         </geometry>
       </collision>
@@ -23,5 +24,5 @@
         <origin xyz="0 0 0" rpy="0 0 0"/>
         <geometry>
-          <mesh filename="package://fanuc_m710ic_support/meshes/m710ic45m/visual/link_1.stl"/>
+          <mesh filename="package://fanuc_m710ic_support/meshes/m710ic50/visual/link_1.stl"/>
         </geometry>
         <xacro:material_fanuc_yellow />
@@ -30,5 +31,5 @@
         <origin xyz="0 0 0" rpy="0 0 0"/>
         <geometry>
-          <mesh filename="package://fanuc_m710ic_support/meshes/m710ic45m/collision/link_1.stl"/>
+          <mesh filename="package://fanuc_m710ic_support/meshes/m710ic50/collision/link_1.stl"/>
         </geometry>
       </collision>
@@ -53,5 +54,5 @@
         <origin xyz="0 0 0" rpy="0 0 0"/>
         <geometry>
-          <mesh filename="package://fanuc_m710ic_support/meshes/m710ic45m/visual/link_3.stl"/>
+          <mesh filename="package://fanuc_m710ic_support/meshes/m710ic50/visual/link_3.stl"/>
         </geometry>
         <xacro:material_fanuc_yellow />
@@ -60,5 +61,5 @@
         <origin xyz="0 0 0" rpy="0 0 0"/>
         <geometry>
-          <mesh filename="package://fanuc_m710ic_support/meshes/m710ic45m/collision/link_3.stl"/>
+          <mesh filename="package://fanuc_m710ic_support/meshes/m710ic50/collision/link_3.stl"/>
         </geometry>
       </collision>
@@ -68,5 +69,5 @@
         <origin xyz="0 0 0" rpy="0 0 0"/>
         <geometry>
-          <mesh filename="package://fanuc_m710ic_support/meshes/m710ic45m/visual/link_4.stl"/>
+          <mesh filename="package://fanuc_m710ic_support/meshes/m710ic50/visual/link_4.stl"/>
         </geometry>
         <xacro:material_fanuc_yellow />
@@ -75,5 +76,5 @@
         <origin xyz="0 0 0" rpy="0 0 0"/>
         <geometry>
-          <mesh filename="package://fanuc_m710ic_support/meshes/m710ic45m/collision/link_4.stl"/>
+          <mesh filename="package://fanuc_m710ic_support/meshes/m710ic50/collision/link_4.stl"/>
         </geometry>
       </collision>
@@ -83,5 +84,5 @@
         <origin xyz="0 0 0" rpy="0 0 0"/>
         <geometry>
-          <mesh filename="package://fanuc_m710ic_support/meshes/m710ic45m/visual/link_5.stl"/>
+          <mesh filename="package://fanuc_m710ic_support/meshes/m710ic50/visual/link_5.stl"/>
         </geometry>
         <xacro:material_fanuc_yellow />
@@ -90,5 +91,5 @@
         <origin xyz="0 0 0" rpy="0 0 0"/>
         <geometry>
-          <mesh filename="package://fanuc_m710ic_support/meshes/m710ic45m/collision/link_5.stl"/>
+          <mesh filename="package://fanuc_m710ic_support/meshes/m710ic50/collision/link_5.stl"/>
         </geometry>
       </collision>
@@ -98,5 +99,5 @@
         <origin xyz="0 0 0" rpy="0 0 0"/>
         <geometry>
-          <mesh filename="package://fanuc_m710ic_support/meshes/m710ic45m/visual/link_6.stl"/>
+          <mesh filename="package://fanuc_m710ic_support/meshes/m710ic50/visual/link_6.stl"/>
         </geometry>
         <xacro:material_fanuc_black />
@@ -105,5 +106,5 @@
         <origin xyz="0 0 0" rpy="0 0 0"/>
         <geometry>
-          <mesh filename="package://fanuc_m710ic_support/meshes/m710ic45m/collision/link_6.stl"/>
+          <mesh filename="package://fanuc_m710ic_support/meshes/m710ic50/collision/link_6.stl"/>
         </geometry>
       </collision>

Commit message: Re-use meshes from M710iC50

File: fanuc_m710ic_support/urdf/m710ic45m_macro.xacro (robot description, xacro)
@@ -2,5 +2,5 @@
 <robot xmlns:xacro="http://wiki.ros.org/xacro">
   <xacro:include filename="$(find fanuc_resources)/urdf/common_materials.xacro"/>
-  <!-- Only link 2 and 4 differ from a M-710iC50 so we re-use them -->
+  <!-- Only links 2 and 4 differ from a M-710iC50 so we re-use them -->
   <xacro:macro name="fanuc_m710ic45m" params="prefix">
     <!-- links: main serial chain -->
@@ -69,5 +69,5 @@
         <origin xyz="0 0 0" rpy="0 0 0"/>
         <geometry>
-          <mesh filename="package://fanuc_m710ic_support/meshes/m710ic50/visual/link_4.stl"/>
+          <mesh filename="package://fanuc_m710ic_support/meshes/m710ic45m/visual/link_4.stl"/>
         </geometry>
         <xacro:material_fanuc_yellow />
@@ -76,5 +76,5 @@
         <origin xyz="0 0 0" rpy="0 0 0"/>
         <geometry>
-          <mesh filename="package://fanuc_m710ic_support/meshes/m710ic50/collision/link_4.stl"/>
+          <mesh filename="package://fanuc_m710ic_support/meshes/m710ic45m/collision/link_4.stl"/>
         </geometry>
       </collision>
