Commit message: Set joint effort for LRMate200iD
based on http://www.fanuc.co.jp/en/product/catalog/pdf/robot/LRMate200iD(E)_v04.pdf

File: fanuc_lrmate200id_support/urdf/lrmate200id_macro.xacro (robot description, xacro)
@@ -115,5 +115,5 @@
       <child link="${prefix}link_1" />
       <axis xyz="0 0 1" />
-      <limit effort="0" lower="-2.965" upper="2.965" velocity="7.85" />
+      <limit effort="16.6" lower="-2.965" upper="2.965" velocity="7.85" />
     </joint>
     <joint name="${prefix}joint_2" type="revolute">
@@ -122,5 +122,5 @@
       <child link="${prefix}link_2" />
       <axis xyz="0 1 0" />
-      <limit effort="0" lower="-1.745329" upper="2.530727" velocity="6.63" />
+      <limit effort="16.6" lower="-1.745329" upper="2.530727" velocity="6.63" />
     </joint>
     <joint name="${prefix}joint_3" type="revolute">
@@ -129,5 +129,5 @@
       <child link="${prefix}link_3" />
       <axis xyz="0 -1 0" />
-      <limit effort="0" lower="-2.450966" upper="4.886922" velocity="9.08" />
+      <limit effort="16.6" lower="-2.450966" upper="4.886922" velocity="9.08" />
     </joint>
     <joint name="${prefix}joint_4" type="revolute">
@@ -136,5 +136,5 @@
       <child link="${prefix}link_4"/>
       <axis xyz="-1 0 0"/>
-      <limit effort="0" lower="-3.315" upper="3.315" velocity="9.60" />
+      <limit effort="16.6" lower="-3.315" upper="3.315" velocity="9.60" />
     </joint>
     <joint name="${prefix}joint_5" type="revolute">
@@ -143,5 +143,5 @@
       <child link="${prefix}link_5"/>
       <axis xyz="0 -1 0"/>
-      <limit effort="0" lower="-2.18" upper="2.18" velocity="9.51" />
+      <limit effort="16.6" lower="-2.18" upper="2.18" velocity="9.51" />
     </joint>
     <joint name="${prefix}joint_6" type="revolute">
@@ -150,5 +150,5 @@
       <child link="${prefix}link_6"/>
       <axis xyz="-1 0 0"/>
-      <limit effort="0" lower="-6.285" upper="6.285" velocity="17.45" />
+      <limit effort="9.4" lower="-6.285" upper="6.285" velocity="17.45" />
     </joint>
     <joint name="${prefix}joint_6-tool0" type="fixed">

Commit message: Set inertial for LRMate200iD for Gazebo simulation

File: fanuc_lrmate200id_support/urdf/lrmate200id_macro.xacro (robot description, xacro)
@@ -18,4 +18,9 @@
         </geometry>
       </collision>
+      <inertial>
+        <origin rpy="0 0 0" xyz="0 0 0"/>
+        <mass value="9"/>
+        <inertia ixx="1.0" ixy="0.0" ixz="0.0" iyy="1.0" iyz="0.0" izz="1.0"/>
+      </inertial>
     </link>
     <link name="${prefix}link_1">
@@ -33,4 +38,9 @@
         </geometry>
       </collision>
+      <inertial>
+        <origin rpy="0 0 0" xyz="0 0 0"/>
+        <mass value="5"/>
+        <inertia ixx="1.0" ixy="0.0" ixz="0.0" iyy="1.0" iyz="0.0" izz="1.0"/>
+      </inertial>
     </link>
     <link name="${prefix}link_2">
@@ -48,4 +58,9 @@
         </geometry>
       </collision>
+      <inertial>
+        <origin rpy="0 0 0" xyz="0 0 0"/>
+        <mass value="4"/>
+        <inertia ixx="1.0" ixy="0.0" ixz="0.0" iyy="1.0" iyz="0.0" izz="1.0"/>
+      </inertial>
     </link>
     <link name="${prefix}link_3">
@@ -63,4 +78,9 @@
         </geometry>
       </collision>
+      <inertial>
+        <origin rpy="0 0 0" xyz="0 0 0"/>
+        <mass value="3"/>
+        <inertia ixx="1.0" ixy="0.0" ixz="0.0" iyy="1.0" iyz="0.0" izz="1.0"/>
+      </inertial>
     </link>
     <link name="${prefix}link_4">
@@ -78,4 +98,9 @@
         </geometry>
       </collision>
+      <inertial>
+        <origin rpy="0 0 0" xyz="0 0 0"/>
+        <mass value="2"/>
+        <inertia ixx="1.0" ixy="0.0" ixz="0.0" iyy="1.0" iyz="0.0" izz="1.0"/>
+      </inertial>
     </link>
     <link name="${prefix}link_5">
@@ -93,4 +118,9 @@
         </geometry>
       </collision>
+      <inertial>
+        <origin rpy="0 0 0" xyz="0 0 0"/>
+        <mass value="1"/>
+        <inertia ixx="1.0" ixy="0.0" ixz="0.0" iyy="1.0" iyz="0.0" izz="1.0"/>
+      </inertial>
     </link>
     <link name="${prefix}link_6">
@@ -108,4 +138,9 @@
         </geometry>
       </collision>
+      <inertial>
+        <origin rpy="0 0 0" xyz="0 0 0"/>
+        <mass value="1"/>
+        <inertia ixx="1.0" ixy="0.0" ixz="0.0" iyy="1.0" iyz="0.0" izz="1.0"/>
+      </inertial>
     </link>
     <link name="${prefix}tool0" />

Commit message: Set joint dynamics 1.0 for gazebo simulation

File: fanuc_lrmate200id_support/urdf/lrmate200id_macro.xacro (robot description, xacro)
@@ -151,4 +151,5 @@
       <axis xyz="0 0 1" />
       <limit effort="0" lower="-2.965" upper="2.965" velocity="7.85" />
+      <dynamics damping="1.0" friction="1.0"/>
     </joint>
     <joint name="${prefix}joint_2" type="revolute">
@@ -158,4 +159,5 @@
       <axis xyz="0 1 0" />
       <limit effort="0" lower="-1.745329" upper="2.530727" velocity="6.63" />
+      <dynamics damping="1.0" friction="1.0"/>
     </joint>
     <joint name="${prefix}joint_3" type="revolute">
@@ -165,4 +167,5 @@
       <axis xyz="0 -1 0" />
       <limit effort="0" lower="-2.450966" upper="4.886922" velocity="9.08" />
+      <dynamics damping="1.0" friction="1.0"/>
     </joint>
     <joint name="${prefix}joint_4" type="revolute">
@@ -172,4 +175,5 @@
       <axis xyz="-1 0 0"/>
       <limit effort="0" lower="-3.315" upper="3.315" velocity="9.60" />
+      <dynamics damping="1.0" friction="1.0"/>
     </joint>
     <joint name="${prefix}joint_5" type="revolute">
@@ -179,4 +183,5 @@
       <axis xyz="0 -1 0"/>
       <limit effort="0" lower="-2.18" upper="2.18" velocity="9.51" />
+      <dynamics damping="1.0" friction="1.0"/>
     </joint>
     <joint name="${prefix}joint_6" type="revolute">
@@ -186,4 +191,5 @@
       <axis xyz="-1 0 0"/>
       <limit effort="0" lower="-6.285" upper="6.285" velocity="17.45" />
+      <dynamics damping="1.0" friction="1.0"/>
     </joint>
     <joint name="${prefix}joint_6-tool0" type="fixed">

Commit message: Define mass parameters as property

File: fanuc_lrmate200id_support/urdf/lrmate200id_macro.xacro (robot description, xacro)
@@ -3,4 +3,12 @@
   <xacro:include filename="$(find fanuc_resources)/urdf/common_materials.xacro"/>
   <xacro:include filename="$(find fanuc_resources)/urdf/common_constants.xacro"/>
+  <!-- Inertia parameters -->
+  <property name="base_link_mass" value="6.215" />  <!-- This mass might be incorrect -->
+  <property name="link_1_mass" value="2.13" />
+  <property name="link_2_mass" value="7.65" />
+  <property name="link_3_mass" value="2.91" />
+  <property name="link_4_mass" value="3.70" />
+  <property name="link_5_mass" value="1.70" />
+  <property name="link_6_mass" value="0.137" />  <!-- This mass might be incorrect -->
   <xacro:macro name="fanuc_lrmate200id" params="prefix">
     <link name="${prefix}base_link">
@@ -20,5 +28,5 @@
       <inertial>
         <origin rpy="0 0 0" xyz="0 0 0"/>
-        <mass value="9"/>
+        <mass value="${base_link_mass}"/>
         <inertia ixx="1.0" ixy="0.0" ixz="0.0" iyy="1.0" iyz="0.0" izz="1.0"/>
       </inertial>
@@ -40,5 +48,5 @@
       <inertial>
         <origin rpy="0 0 0" xyz="0 0 0"/>
-        <mass value="5"/>
+        <mass value="${link_1_mass}"/>
         <inertia ixx="1.0" ixy="0.0" ixz="0.0" iyy="1.0" iyz="0.0" izz="1.0"/>
       </inertial>
@@ -60,5 +68,5 @@
       <inertial>
         <origin rpy="0 0 0" xyz="0 0 0"/>
-        <mass value="4"/>
+        <mass value="${link_2_mass}"/>
         <inertia ixx="1.0" ixy="0.0" ixz="0.0" iyy="1.0" iyz="0.0" izz="1.0"/>
       </inertial>
@@ -80,5 +88,5 @@
       <inertial>
         <origin rpy="0 0 0" xyz="0 0 0"/>
-        <mass value="3"/>
+        <mass value="${link_3_mass}"/>
         <inertia ixx="1.0" ixy="0.0" ixz="0.0" iyy="1.0" iyz="0.0" izz="1.0"/>
       </inertial>
@@ -100,5 +108,5 @@
       <inertial>
         <origin rpy="0 0 0" xyz="0 0 0"/>
-        <mass value="2"/>
+        <mass value="${link_4_mass}"/>
         <inertia ixx="1.0" ixy="0.0" ixz="0.0" iyy="1.0" iyz="0.0" izz="1.0"/>
       </inertial>
@@ -120,5 +128,5 @@
       <inertial>
         <origin rpy="0 0 0" xyz="0 0 0"/>
-        <mass value="1"/>
+        <mass value="${link_5_mass}"/>
         <inertia ixx="1.0" ixy="0.0" ixz="0.0" iyy="1.0" iyz="0.0" izz="1.0"/>
       </inertial>
@@ -140,5 +148,5 @@
       <inertial>
         <origin rpy="0 0 0" xyz="0 0 0"/>
-        <mass value="1"/>
+        <mass value="${link_6_mass}"/>
         <inertia ixx="1.0" ixy="0.0" ixz="0.0" iyy="1.0" iyz="0.0" izz="1.0"/>
       </inertial>

Commit message: Compute inertia values with meshlab

File: fanuc_lrmate200id_support/urdf/lrmate200id_macro.xacro (robot description, xacro)
@@ -27,7 +27,8 @@
       </collision>
       <inertial>
-        <origin rpy="0 0 0" xyz="0 0 0"/>
+        <origin xyz="0 0 0" rpy="0 0 0"/>
         <mass value="${base_link_mass}"/>
-        <inertia ixx="1.0" ixy="0.0" ixz="0.0" iyy="1.0" iyz="0.0" izz="1.0"/>
+        <!-- Copied from abb_irb120t https://github.com/ros-industrial/abb_experimental/blob/indigo-devel/abb_irb120_support/urdf/irb120t_macro.xacro. -->
+        <inertia ixx="0.0247272" ixy="-8.0784E-05" ixz="0.00130902" iyy="0.0491285" iyz="-8.0419E-06" izz="0.0472376"/>
       </inertial>
     </link>
@@ -47,7 +48,11 @@
       </collision>
       <inertial>
-        <origin rpy="0 0 0" xyz="0 0 0"/>
+        <origin xyz="-0.000010 -0.054550 0.028725" rpy="0 0 0"/>
         <mass value="${link_1_mass}"/>
-        <inertia ixx="1.0" ixy="0.0" ixz="0.0" iyy="1.0" iyz="0.0" izz="1.0"/>
+        <!-- Estimated with Meshlab and stl model. '600' is the scale to make inertial to be standard values
+             refering abb_irb120t https://github.com/ros-industrial/abb_experimental/blob/indigo-devel/abb_irb120_support/urdf/irb120t_macro.xacro. -->
+        <inertia
+          ixx="${600 * 0.000048}" ixy="0.0" ixz="${600 * -0.000006}"
+          iyy="${600 * 0.000035}" iyz="0.0" izz="${600 * 0.000037}"/>
       </inertial>
     </link>
@@ -67,7 +72,10 @@
       </collision>
       <inertial>
-        <origin rpy="0 0 0" xyz="0 0 0"/>
+        <origin xyz="-0.002701 -0.000977 0.159466" rpy="0 0 0"/>
         <mass value="${link_2_mass}"/>
-        <inertia ixx="1.0" ixy="0.0" ixz="0.0" iyy="1.0" iyz="0.0" izz="1.0"/>
+        <inertia
+          ixx="${600 * 0.000182}" ixy="0.0" ixz="0.0"
+          iyy="${600 * 0.000157}" iyz="${600 * -0.000001}"
+          izz="${600 * 0.000049}"/>
       </inertial>
     </link>
@@ -87,7 +95,10 @@
       </collision>
       <inertial>
-        <origin rpy="0 0 0" xyz="0 0 0"/>
+        <origin xyz="-0.000065 0.017074 0.008866" rpy="0 0 0"/>
         <mass value="${link_3_mass}"/>
-        <inertia ixx="1.0" ixy="0.0" ixz="0.0" iyy="1.0" iyz="0.0" izz="1.0"/>
+        <inertia
+          ixx="${600 * 0.000007}" ixy="0.0" ixz="${600 * -0.000001}"
+          iyy="${600 * 0.000008}" iyz="0.0"
+          izz="${600 * 0.000008}"/>
       </inertial>
     </link>
@@ -107,7 +118,10 @@
       </collision>
       <inertial>
-        <origin rpy="0 0 0" xyz="0 0 0"/>
+        <origin xyz="0.000067 0.002203 0.221634" rpy="0 0 0"/>
         <mass value="${link_4_mass}"/>
-        <inertia ixx="1.0" ixy="0.0" ixz="0.0" iyy="1.0" iyz="0.0" izz="1.0"/>
+        <inertia
+          ixx="${600 * 0.000005}" ixy="0.0" ixz="0.0"
+          iyy="${600 * 0.000019}" iyz="0.0"
+          izz="${600 * 0.000019}"/>
       </inertial>
     </link>
@@ -127,7 +141,11 @@
       </collision>
       <inertial>
-        <origin rpy="0 0 0" xyz="0 0 0"/>
+        <origin xyz="-0.000010 -0.054550 0.028725" rpy="0 0 0"/>
         <mass value="${link_5_mass}"/>
-        <inertia ixx="1.0" ixy="0.0" ixz="0.0" iyy="1.0" iyz="0.0" izz="1.0"/>
+        <!-- This mass might be incorrect because of nan value of
+             'link_5.stl' in Meshlab inertia estimation. -->
+        <inertia
+          ixx="${600 * 0.00004}" ixy="0.0" ixz="${600 * -0.000004}"
+          iyy="${600 * 0.00003}" iyz="0.0" izz="${600 * 0.00003}"/>
       </inertial>
     </link>
@@ -147,7 +165,10 @@
       </collision>
       <inertial>
-        <origin rpy="0 0 0" xyz="0 0 0"/>
+        <origin xyz="-0.000000 0.000000 -0.003006" rpy="0 0 0" />
         <mass value="${link_6_mass}"/>
-        <inertia ixx="1.0" ixy="0.0" ixz="0.0" iyy="1.0" iyz="0.0" izz="1.0"/>
+        <inertia
+          ixx="0.01" ixy="0.0" ixz="0.0"
+          iyy="0.01" iyz="0.0"
+          izz="0.01"/>
       </inertial>
     </link>

Commit message: gazebo: integration of gazebo sim for lrmate200id

File: fanuc_lrmate200id_support/urdf/lrmate200id_macro.xacro (robot description, xacro)
@@ -1,4 +1,4 @@
 <?xml version="1.0"?>
-<robot xmlns:xacro="http://wiki.ros.org/xacro">
+<robot xmlns:xacro="http://www.ros.org/wiki/xacro">
   <xacro:include filename="$(find fanuc_resources)/urdf/common_materials.xacro"/>
   <xacro:macro name="fanuc_lrmate200id" params="prefix">
@@ -116,6 +116,7 @@
       <axis xyz="0 0 1" />
       <limit effort="0" lower="-2.965" upper="2.965" velocity="7.85" />
-    </joint>
-    <joint name="${prefix}joint_2" type="revolute">
+      <dynamics damping="0.0" friction="0.0"/>
+   </joint>
+   <joint name="${prefix}joint_2" type="revolute">
       <origin xyz="0.050 0 0" rpy="0 0 0"/>
       <parent link="${prefix}link_1" />
