Commit message: fix path to stl files

File: fanuc_lrmate200id_support/urdf/gripper_macro.xacro (robot description, xacro)
@@ -2,169 +2,176 @@
 <robot xmlns:xacro="http://www.ros.org/wiki/xacro">
 <xacro:macro name="gripper" params="prefix">
-<xacro:include filename="$(find fanuc_resources)/urdf/common_materials.xacro"/>
-<!-- Part 6 Gripper Base Joint -->
-<joint name = "Part6_Gripper_Base" type="revolute">
-	<parent link="tool0"/>
-	<child link ="Gripper_Base"/>
-	<origin xyz="0 0 0" rpy="0 3.14 0"/>
-	<axis xyz="0 0 1"/>
-	<dynamics damping="0.7"/>
-	<limit effort="100" lower="-0.5232" upper="0.5232" velocity="100"/>
-</joint>
-<!-- Gripper Base -->
-<link name="Gripper_Base">
-	<collision>
-		<origin xyz="-0.065 -0.065 0" rpy ="-1.57 0 0"/>
-		<geometry>
-			<mesh filename="package://fanuc_lrmate200id_support/meshes/Gripper_base.STL" scale="0.001 0.001 0.001"/>
-		</geometry>
-	</collision>
-	<visual>
-		<origin xyz="-0.065 -0.065 0" rpy ="-1.57 0 0"/>
-		<geometry>
-			<mesh filename="package://fanuc_lrmate200id_support/meshes/Gripper_base.STL" scale="0.001 0.001 0.001"/>
-		</geometry>
-        <xacro:material_fanuc_yellow />
-	</visual>
-	<inertial>
-		<origin xyz = "0.00112 0.04196 0" rpy ="0 0 0"/>
-		<mass value = "1.067"/>
-		<inertia ixx ="0.00372062398" iyy=".00223540544" izz=".003641916" ixy="-0.000013337910" ixz ="0.000000013" iyz = "-0.00000003496"/>
-	</inertial>
-</link>
-<gazebo reference= "Gripper_Base" >
-	<material>Gazebo/Black</material>
-</gazebo>
-<!-- Gripper Base Finger 3 Joint-->
-<joint name = "Gripper_Finger3" type="revolute">
-	<parent link="Gripper_Base"/>
-	<child link ="Finger3"/>
-	<origin xyz="0.04448 0 -0.09533" rpy="0 0 0"/>
-	<axis xyz="0 1 0"/>
-	<dynamics damping="0.7"/>
-	<limit effort="1" lower="-0.0872" upper="0.0872" velocity="6.1087"/>
-</joint>
-<!-- Finger 3-->
-<link name="Finger3">
-	<collision>
-		<origin xyz="0.075 0.038 0.075" rpy ="-1.57 0 3.14"/>
-		<geometry>
-			<mesh filename="package://fanuc_lrmate200id_support/meshes/Gripper_finger.STL" scale="0.001 0.001 0.001"/>
-		</geometry>
-	</collision>
-	<visual>
-		<origin xyz="0.075 0.038 0.075" rpy ="-1.57 0 3.14"/>
-		<geometry>
-			<mesh filename="package://fanuc_lrmate200id_support/meshes/Gripper_finger.STL" scale="0.001 0.001 0.001"/>
-		</geometry>
-	    <xacro:material_fanuc_gray28 />
-	</visual>
-	<inertial>
-		<origin xyz = "0.00112 0.04196 0" rpy ="0 0 0"/>
-		<mass value = "0.17495"/>
-		<inertia ixx ="0.002449587" iyy=".00018834795" izz=".00315304482" ixy="-0.00141880714" ixz ="-0.00044070839" iyz = "-0.00067806067"/>
-	</inertial>
-</link>
-<!-- Base Finger1 Joint -->
-<!-- Gripper Base Finger 1 Joint-->
-<joint name = "Gripper_Finger1" type="revolute">
-	<parent link="Gripper_Base"/>
-	<child link ="Finger1"/>
-	<origin xyz="-0.04448 0.04 -0.09533" rpy="0 0 0"/>
-	<axis xyz="0 1 0"/>
-	<dynamics damping="0.7"/>
-	<limit effort="1" lower="-0.0872" upper="0.0872" velocity="6.1087"/>
-</joint>
-<!-- Finger 1-->
-<link name="Finger1">
-	<collision>
-		<origin xyz="-0.075 -0.038 0.075" rpy ="-1.57 0 0"/>
-		<geometry>
-			<mesh filename="package://fanuc_lrmate200id_support/meshes/Gripper_finger.STL" scale="0.001 0.001 0.001"/>
-		</geometry>
-	</collision>
-	<visual>
-		<origin xyz="-0.075 -0.038 0.075" rpy ="-1.57 0 0"/>
-		<geometry>
-			<mesh filename="package://fanuc_lrmate200id_support/meshes/Gripper_finger.STL" scale="0.001 0.001 0.001"/>
-		</geometry>
-        <xacro:material_fanuc_gray28 />
-	</visual>
-	<inertial>
-		<origin xyz = "0.00112 0.04196 0" rpy ="0 0 0"/>
-		<mass value = "0.17495"/>
-		<inertia ixx ="0.002449587" iyy=".00018834795" izz=".00315304482" ixy="-0.00141880714" ixz ="-0.00044070839" iyz = "-0.00067806067"/>
-	</inertial>
-</link>
-<!-- Gripper Base Finger 2 Joint-->
-<joint name = "Gripper_Finger2" type="revolute">
-	<parent link="Gripper_Base"/>
-	<child link ="Finger2"/>
-	<origin xyz="-0.04448 -0.04 -0.09533" rpy="0 0 0"/>
-	<axis xyz="0 1 0"/>
-	<dynamics damping="0.7"/>
-	<limit effort="1" lower="-0.0872" upper="0.0872" velocity="6.1087"/>
-</joint>
-<!-- Finger 2-->
-<link name="Finger2">
-	<collision>
-		<origin xyz="-0.075 -0.038 0.075" rpy ="-1.57 0 0"/>
-		<geometry>
-			<mesh filename="package://fanuc_lrmate200id_support/meshes/Gripper_finger.STL" scale="0.001 0.001 0.001"/>
-		</geometry>
-	</collision>
-	<visual>
-		<origin xyz="-0.075 -0.038 0.075" rpy ="-1.57 0 0"/>
-		<geometry>
-			<mesh filename="package://fanuc_lrmate200id_support/meshes/Gripper_finger.STL" scale="0.001 0.001 0.001"/>
-		</geometry>
-        <xacro:material_fanuc_gray28 />
-	</visual>
-	<inertial>
-		<origin xyz = "0.00112 0.04196 0" rpy ="0 0 0"/>
-		<mass value = "0.17495"/>
-		<inertia ixx ="0.002449587" iyy=".00018834795" izz=".00315304482" ixy="-0.00141880714" ixz ="-0.00044070839" iyz = "-0.00067806067"/>
-	</inertial>
-</link>
-<transmission name="tran6">
-    <type>transmission_interface/SimpleTransmission</type>
-    <joint name="Part6_Gripper_Base">
-      <hardwareInterface>PositionJointInterface</hardwareInterface>
+    <!-- Part 6 Gripper Base Joint -->
+    <joint name="Part6_Gripper_Base" type="revolute">
+        <parent link="link_6" />
+        <child link="Gripper_Base" />
+        <origin rpy="0 -1.57 0" xyz="0 0 0" />
+        <axis xyz="0 0 1" />
+        <dynamics damping="0.7" />
+        <limit effort="100" lower="-0.5232" upper="0.5232" velocity="100" />
     </joint>
-    <actuator name="Part6_Gripper_Base_motor">
-      <hardwareInterface>PositionJointInterface</hardwareInterface>
-      <mechanicalReduction>1</mechanicalReduction>
-    </actuator>
-  </transmission>
- <transmission name="tran7">
-    <type>transmission_interface/SimpleTransmission</type>
-    <joint name="Gripper_Finger3">
-      <hardwareInterface>PositionJointInterface</hardwareInterface>
+    <!-- Gripper Base -->
+    <link name="Gripper_Base">
+        <collision>
+            <origin rpy="-1.57 0 0" xyz="-0.065 -0.065 0" />
+            <geometry>
+                <mesh filename="package://fanuc_lrmate200id_support/meshes/gripper/collision/Gripper_base.STL" scale="0.001 0.001 0.001" />
+            </geometry>
+        </collision>
+        <visual>
+            <origin rpy="-1.57 0 0" xyz="-0.065 -0.065 0" />
+            <geometry>
+                <mesh filename="package://fanuc_lrmate200id_support/meshes/gripper/visual/Gripper_base.STL" scale="0.001 0.001 0.001" />
+            </geometry>
+            <material name="">
+                <color rgba="0.96 0.76 0.13 1.0" />
+            </material>
+        </visual>
+<inertial>
+            <origin rpy="0 0 0" xyz="0.00112 0.04196 0" />
+            <mass value="1.067" />
+            <inertia ixx="0.00372062398" ixy="-0.000013337910" ixz="0.000000013" iyy=".00223540544" iyz="-0.00000003496" izz=".003641916" />
+        </inertial>
+    </link>
+    <gazebo reference="Gripper_Base">
+        <material>Gazebo/Black</material>
+    </gazebo>
+    <!-- Gripper Base Finger 3 Joint-->
+    <joint name="Gripper_Finger3" type="revolute">
+        <parent link="Gripper_Base" />
+        <child link="Finger3" />
+        <origin rpy="0 0 0" xyz="0.04448 0 -0.09533" />
+        <axis xyz="0 1 0" />
+        <dynamics damping="0.7" />
+        <limit effort="1" lower="-0.0872" upper="0.0872" velocity="6.1087" />
     </joint>
-    <actuator name="Gripper_Finger3_motor">
-      <hardwareInterface>PositionJointInterface</hardwareInterface>
-      <mechanicalReduction>1</mechanicalReduction>
-    </actuator>
-  </transmission>
- <transmission name="tran8">
-    <type>transmission_interface/SimpleTransmission</type>
-    <joint name="Gripper_Finger1">
-      <hardwareInterface>PositionJointInterface</hardwareInterface>
+    <!-- Finger 3-->
+    <link name="Finger3">
+        <collision>
+            <origin rpy="-1.57 0 3.14" xyz="0.075 0.038 0.075" />
+            <geometry>
+                <mesh filename="package://fanuc_lrmate200id_support/meshes/gripper/collision/Gripper_finger.STL" scale="0.001 0.001 0.001" />
+            </geometry>
+        </collision>
+        <visual>
+            <origin rpy="-1.57 0 3.14" xyz="0.075 0.038 0.075" />
+            <geometry>
+                <mesh filename="package://fanuc_lrmate200id_support/meshes/gripper/visual/Gripper_finger.STL" scale="0.001 0.001 0.001" />
+            </geometry>
+            <material name="">
+                <color rgba="0.278431372549 0.278431372549 0.278431372549 1.0" />
+            </material>
+        </visual>
+<inertial>
+            <origin rpy="0 0 0" xyz="0.00112 0.04196 0" />
+            <mass value="0.17495" />
+            <inertia ixx="0.002449587" ixy="-0.00141880714" ixz="-0.00044070839" iyy=".00018834795" iyz="-0.00067806067" izz=".00315304482" />
+        </inertial>
+    </link>
+    <!-- Base Finger1 Joint -->
+    <!-- Gripper Base Finger 1 Joint-->
+    <joint name="Gripper_Finger1" type="revolute">
+        <parent link="Gripper_Base" />
+        <child link="Finger1" />
+        <origin rpy="0 0 0" xyz="-0.04448 0.04 -0.09533" />
+        <axis xyz="0 1 0" />
+        <dynamics damping="0.7" />
+        <limit effort="1" lower="-0.0872" upper="0.0872" velocity="6.1087" />
     </joint>
-    <actuator name="Gripper_Finger1_motor">
-      <hardwareInterface>PositionJointInterface</hardwareInterface>
-      <mechanicalReduction>1</mechanicalReduction>
-    </actuator>
-  </transmission>
- <transmission name="tran9">
-    <type>transmission_interface/SimpleTransmission</type>
-    <joint name="Gripper_Finger2">
-      <hardwareInterface>PositionJointInterface</hardwareInterface>
+    <!-- Finger 1-->
+    <link name="Finger1">
+        <collision>
+            <origin rpy="-1.57 0 0" xyz="-0.075 -0.038 0.075" />
+            <geometry>
+                <mesh filename="package://fanuc_lrmate200id_support/meshes/gripper/collision/Gripper_finger.STL" scale="0.001 0.001 0.001" />
+            </geometry>
+        </collision>
+        <visual>
+            <origin rpy="-1.57 0 0" xyz="-0.075 -0.038 0.075" />
+            <geometry>
+                <mesh filename="package://fanuc_lrmate200id_support/meshes/gripper/visual/Gripper_finger.STL" scale="0.001 0.001 0.001" />
+            </geometry>
+            <material name="">
+                <color rgba="0.278431372549 0.278431372549 0.278431372549 1.0" />
+            </material>
+        </visual>
+<inertial>
+            <origin rpy="0 0 0" xyz="0.00112 0.04196 0" />
+            <mass value="0.17495" />
+            <inertia ixx="0.002449587" ixy="-0.00141880714" ixz="-0.00044070839" iyy=".00018834795" iyz="-0.00067806067" izz=".00315304482" />
+        </inertial>
+    </link>
+    <!-- Gripper Base Finger 2 Joint-->
+    <joint name="Gripper_Finger2" type="revolute">
+        <parent link="Gripper_Base" />
+        <child link="Finger2" />
+        <origin rpy="0 0 0" xyz="-0.04448 -0.04 -0.09533" />
+        <axis xyz="0 1 0" />
+        <dynamics damping="0.7" />
+        <limit effort="1" lower="-0.0872" upper="0.0872" velocity="6.1087" />
     </joint>
-    <actuator name="Gripper_Finger2_motor">
-      <hardwareInterface>PositionJointInterface</hardwareInterface>
-      <mechanicalReduction>1</mechanicalReduction>
-    </actuator>
-  </transmission>
+    <!-- Finger 2-->
+    <link name="Finger2">
+        <collision>
+            <origin rpy="-1.57 0 0" xyz="-0.075 -0.038 0.075" />
+            <geometry>
+                <mesh filename="package://fanuc_lrmate200id_support/meshes/gripper/collision/Gripper_finger.STL" scale="0.001 0.001 0.001" />
+            </geometry>
+        </collision>
+        <visual>
+            <origin rpy="-1.57 0 0" xyz="-0.075 -0.038 0.075" />
+            <geometry>
+                <mesh filename="package://fanuc_lrmate200id_support/meshes/gripper/visual/Gripper_finger.STL" scale="0.001 0.001 0.001" />
+            </geometry>
+            <material name="">
+                <color rgba="0.278431372549 0.278431372549 0.278431372549 1.0" />
+            </material>
+        </visual>
+<inertial>
+            <origin rpy="0 0 0" xyz="0.00112 0.04196 0" />
+            <mass value="0.17495" />
+            <inertia ixx="0.002449587" ixy="-0.00141880714" ixz="-0.00044070839" iyy=".00018834795" iyz="-0.00067806067" izz=".00315304482" />
+        </inertial>
+    </link>
+    <transmission name="trans_Part6_Gripper_Base">
+        <type>transmission_interface/SimpleTransmission</type>
+        <joint name="Part6_Gripper_Base">
+            <hardwareInterface>hardware_interface/PositionJointInterface</hardwareInterface>
+        </joint>
+        <actuator name="Part6_Gripper_Base_motor">
+            <hardwareInterface>hardware_interface/PositionJointInterface</hardwareInterface>
+            <mechanicalReduction>1</mechanicalReduction>
+        </actuator>
+    </transmission>
+    <transmission name="trans_Gripper_Finger3">
+        <type>transmission_interface/SimpleTransmission</type>
+        <joint name="Gripper_Finger3">
+            <hardwareInterface>hardware_interface/PositionJointInterface</hardwareInterface>
+        </joint>
+        <actuator name="Gripper_Finger3_motor">
+            <hardwareInterface>hardware_interface/PositionJointInterface</hardwareInterface>
+            <mechanicalReduction>1</mechanicalReduction>
+        </actuator>
+    </transmission>
+    <transmission name="trans_Gripper_Finger1">
+        <type>transmission_interface/SimpleTransmission</type>
+        <joint name="Gripper_Finger1">
+            <hardwareInterface>hardware_interface/PositionJointInterface</hardwareInterface>
+        </joint>
+        <actuator name="Gripper_Finger1_motor">
+            <hardwareInterface>hardware_interface/PositionJointInterface</hardwareInterface>
+            <mechanicalReduction>1</mechanicalReduction>
+        </actuator>
+    </transmission>
+    <transmission name="trans_Gripper_Finger2">
+        <type>transmission_interface/SimpleTransmission</type>
+        <joint name="Gripper_Finger2">
+            <hardwareInterface>hardware_interface/PositionJointInterface</hardwareInterface>
+        </joint>
+        <actuator name="Gripper_Finger2_motor">
+            <hardwareInterface>hardware_interface/PositionJointInterface</hardwareInterface>
+            <mechanicalReduction>1</mechanicalReduction>
+        </actuator>
+    </transmission>
 	</xacro:macro>
 </robot>
