Commit message: add camera_link

File: fanuc_lrmate200id_support/urdf/lrmate200id7l.xacro (robot description, xacro)
@@ -5,3 +5,11 @@
   <xacro:fanuc_lrmate200id7l prefix=""/>
   <xacro:gripper prefix=""/>
+      <!-- Part 6 Gripper Base Joint -->
+<joint name="camera_joint" type="fixed">
+    <parent link="link_6" />
+    <child link="camera_link" />
+    <origin rpy="3.14 -1.57 0" xyz="0.0 0.0 0.0" />
+    <axis xyz="0 0 0" />
+</joint>
+<link name="camera_link"/>
 </robot>

Commit message: calibrate extrinstic camera params

File: fanuc_lrmate200id_support/urdf/lrmate200id7l.xacro (robot description, xacro)
@@ -7,7 +7,8 @@
       <!-- Part 6 Gripper Base Joint -->
 <joint name="camera_joint" type="fixed">
-    <parent link="link_6" />
+    <parent link="link_4" />
     <child link="camera_link" />
-    <origin rpy="3.14 -1.57 0" xyz="0.0 0.0 0.0" />
+    <origin rpy="-0.0 1.50293 -0.06822"
+     xyz="0.32704 0.02164 -0.07475" />
     <axis xyz="0 0 0" />
 </joint>

Commit message: recalibrate camera

File: fanuc_lrmate200id_support/urdf/lrmate200id7l.xacro (robot description, xacro)
@@ -7,6 +7,6 @@
     <parent link="link_4" />
     <child link="camera_link" />
-    <origin rpy="-0.0 1.50293 -0.06822"
-     xyz="0.32704 0.02164 -0.07475" />
+    <origin rpy="-0.0037 1.50600 -0.0031"
+     xyz="0.32273 0.01841 -0.06556" />
     <axis xyz="0 0 0" />
 </joint>
