Commit message: set correct inertias for lrmate200id and  7l

File: fanuc_lrmate200id_gazebo/urdf/lrmate200id7l_gazebo_macro.xacro (robot description, xacro)
@@ -15,5 +15,5 @@
 			<mesh filename = "package://fanuc_lrmate200id_support/meshes/lrmate200id/collision/base_link.stl"  />
 		</geometry>
-	<origin xyz = "0 0 0" rpy = "0 0 0"/><!-- Best value <origin xyz = "0.105 0.09 0" rpy = "0 0 0" />-->
+	<origin xyz = "0 0 0" rpy = "0 0 0"/>
 	</collision>
 	<visual>
@@ -21,11 +21,10 @@
 			<mesh filename = "package://fanuc_lrmate200id_support/meshes/lrmate200id/visual/base_link.stl" />
 		</geometry>
-	<origin xyz = "0 0 0" rpy = "0 0 0"/><!-- Best value <origin xyz = "0.105 0.09 0" rpy = "0 0 0" />-->
-	</visual>
-	<inertial>
-		<origin xyz = "0.105 0.09 0.08042" rpy = "0 0 0" /> <!-- Best value <origin xyz = "0.105 0.09 0.08042" rpy = "0 0 0" />-->
-		<mass value = "4.85331"/>
-		<inertia ixx ="0.000533781" iyy=".055445798" izz=".02302818052" ixy="0.00012915752" ixz ="-0.002807595" iyz = "-0.000094967"/>
-	</inertial>
+	<origin xyz = "0 0 0" rpy = "0 0 0"/>
+	</visual>
+	<inertial>
+		<origin xyz = "0.0 0.0 0.0" rpy = "0 0 0" />
+		<mass value = "6.215"/>
+        <inertia ixx="0.0247272" ixy="-8.0784E-05" ixz="0.00130902" iyy="0.0491285" iyz="-8.0419E-06" izz="0.0472376"/>	</inertial>
 </link>
 <link name = "world"/>
@@ -44,7 +43,7 @@
       <axis xyz="0 0 1" />
       <limit effort="0" lower="-2.965" upper="2.965" velocity="7.85" />
-</joint>
-<!-- Part 2 -->
-<link name ="${prefix}link_1">
+      <dynamics damping="1.0" friction="1.0"/>
+</joint>
+ <link name ="${prefix}link_1">
 	<collision>
 	<geometry>
@@ -60,8 +59,9 @@
 	</visual>
 	<inertial>
-		<origin xyz = "0.0 0.0 0.081" rpy = "0 0 0" />
-		<mass value = "4.85331"/>
-		<inertia ixx ="0.000533781" iyy=".055445798" izz=".02302818052" ixy="0.00012915752" ixz ="-0.002807595" iyz = "-0.000094967"/>
-	</inertial>
+        <origin xyz="-0.000010 -0.054550 0.028725" rpy="0 0 0"/>
+		<mass value = "2.13"/>
+        <inertia
+          ixx="${600 * 0.000048}" ixy="0.0" ixz="${600 * -0.000006}"
+          iyy="${600 * 0.000035}" iyz="0.0" izz="${600 * 0.000037}"/>	</inertial>
 </link>
 <gazebo reference= "${prefix}link_1" >
@@ -74,4 +74,5 @@
       <axis xyz="0 1 0" />
       <limit effort="0" lower="-1.745329" upper="2.530727" velocity="6.63" />
+      <dynamics damping="1.0" friction="1.0"/>
 </joint>
 <!--Part3-->
@@ -90,8 +91,10 @@
 	</visual>
 	<inertial>
-		<origin xyz = "0 -0.00155 0.17556" rpy ="0 0 0"/>
-		<mass value = "7.96646"/>
-		<inertia ixx ="0.44125720672" iyy=".42103008445" izz=".03658588308" ixy="0.000023323" ixz ="-0.01624821395" iyz = "-0.00127983617"/>
-	</inertial>
+        <origin xyz="-0.002701 -0.000977 0.159466" rpy="0 0 0"/>
+		<mass value = "7.65"/>
+        <inertia
+          ixx="${600 * 0.000182}" ixy="0.0" ixz="0.0"
+          iyy="${600 * 0.000157}" iyz="${600 * -0.000001}"
+          izz="${600 * 0.000049}"/>	</inertial>
 </link>
 <gazebo reference= "${prefix}link_2" >
@@ -104,4 +107,5 @@
       <axis xyz="0 -1 0" />
       <limit effort="0" lower="-2.450966" upper="4.886922" velocity="9.08" />
+      <dynamics damping="1.0" friction="1.0"/>
 </joint>
 <link name="${prefix}link_3">
@@ -119,8 +123,10 @@
 	</visual>
 	<inertial>
-		<origin xyz = "0.008 0.00068 0.0177" rpy ="0 0 0"/>
-		<mass value = "2.401"/>
-		<inertia ixx ="0.00709493364" iyy=".08303386" izz=".007482747" ixy="0.000062924" ixz ="0.000131383" iyz = "0.000095227"/>
-	</inertial>
+        <origin xyz="-0.000065 0.017074 0.008866" rpy="0 0 0"/>
+		<mass value = "2.91"/>
+        <inertia
+          ixx="${600 * 0.000007}" ixy="0.0" ixz="${600 * -0.000001}"
+          iyy="${600 * 0.000008}" iyz="0.0"
+          izz="${600 * 0.000008}"/>	</inertial>
 </link>
 <gazebo reference= "${prefix}link_3" >
@@ -133,4 +139,5 @@
       <axis xyz="-1 0 0"/>
       <limit effort="0" lower="-3.315" upper="3.315" velocity="9.60" />
+      <dynamics damping="1.0" friction="1.0"/>
 </joint>
 <link name="${prefix}link_4">
@@ -148,8 +155,10 @@
 	</visual>
 	<inertial>
-		<origin xyz = "0.24013 0 0" rpy ="0 0 0"/>
-		<mass value = "2.89084"/>
-		<inertia ixx ="0.004863267" iyy=".19336297539" izz=".19385148073" ixy="0.00303203667" ixz ="0.000018846079" iyz = "-0.00000096841"/>
-	</inertial>
+        <origin xyz="0.000067 0.002203 0.221634" rpy="0 0 0"/>
+		<mass value = "3.70"/>
+        <inertia
+          ixx="${600 * 0.000005}" ixy="0.0" ixz="0.0"
+          iyy="${600 * 0.000019}" iyz="0.0"
+          izz="${600 * 0.000019}"/>	</inertial>
 </link>
 <gazebo reference= "${prefix}link_4" >
@@ -162,4 +171,5 @@
       <axis xyz="0 -1 0"/>
       <limit effort="0" lower="-2.18" upper="2.18" velocity="9.51" />
+	  <dynamics damping="1.0" friction="1.0"/>
 </joint>
 <link name="${prefix}link_5">
@@ -177,8 +187,9 @@
 	</visual>
 	<inertial>
-		<origin xyz = "0.01573 0.003 -0.00006" rpy ="0 0 0"/>
-		<mass value = "0.043284"/>
-		<inertia ixx ="0.00029985018" iyy=".000661879" izz=".00064231094" ixy="-0.00000439197" ixz ="-0.000000345" iyz = "-0.00000008651"/>
-	</inertial>
+        <origin xyz="-0.000010 -0.054550 0.028725" rpy="0 0 0"/>
+		<mass value = "1.70"/>
+        <inertia
+          ixx="${600 * 0.00004}" ixy="0.0" ixz="${600 * -0.000004}"
+          iyy="${600 * 0.00003}" iyz="0.0" izz="${600 * 0.00003}"/>	</inertial>
 </link>
 <gazebo reference= "${prefix}link_5" >
@@ -191,4 +202,5 @@
       <axis xyz="-1 0 0"/>
       <limit effort="0" lower="-6.285" upper="6.285" velocity="17.45" />
+	  <dynamics damping="1.0" friction="1.0"/>
 </joint>
 <link name="${prefix}link_6">
@@ -206,7 +218,10 @@
 	</visual>
 	<inertial>
-		<origin xyz = "0.01573 0.003 -0.00006" rpy ="0 0 0"/>
-		<mass value = "0.043284"/>
-		<inertia ixx ="0.00029985018" iyy=".000661879" izz=".00064231094" ixy="-0.00000439197" ixz ="-0.000000345" iyz = "-0.00000008651"/>
+        <origin xyz="-0.000000 0.000000 -0.003006" rpy="0 0 0" />
+		<mass value = "0.137"/>
+        <inertia
+          ixx="0.01" ixy="0.0" ixz="0.0"
+          iyy="0.01" iyz="0.0"
+          izz="0.01"/>
 	</inertial>
 </link>

File: fanuc_lrmate200id_gazebo/urdf/lrmate200id_gazebo_macro.xacro (robot description, xacro)
@@ -15,5 +15,5 @@
 			<mesh filename = "package://fanuc_lrmate200id_support/meshes/lrmate200id/collision/base_link.stl"  />
 		</geometry>
-	<origin xyz = "0 0 0" rpy = "0 0 0"/><!-- Best value <origin xyz = "0.105 0.09 0" rpy = "0 0 0" />-->
+	<origin xyz = "0 0 0" rpy = "0 0 0"/>
 	</collision>
 	<visual>
@@ -21,11 +21,10 @@
 			<mesh filename = "package://fanuc_lrmate200id_support/meshes/lrmate200id/visual/base_link.stl" />
 		</geometry>
-	<origin xyz = "0 0 0" rpy = "0 0 0"/><!-- Best value <origin xyz = "0.105 0.09 0" rpy = "0 0 0" />-->
-	</visual>
-	<inertial>
-		<origin xyz = "0.105 0.09 0.08042" rpy = "0 0 0" /> <!-- Best value <origin xyz = "0.105 0.09 0.08042" rpy = "0 0 0" />-->
-		<mass value = "4.85331"/>
-		<inertia ixx ="0.000533781" iyy=".055445798" izz=".02302818052" ixy="0.00012915752" ixz ="-0.002807595" iyz = "-0.000094967"/>
-	</inertial>
+	<origin xyz = "0 0 0" rpy = "0 0 0"/>
+	</visual>
+	<inertial>
+		<origin xyz = "0.0 0.0 0.0" rpy = "0 0 0" />
+		<mass value = "6.215"/>
+        <inertia ixx="0.0247272" ixy="-8.0784E-05" ixz="0.00130902" iyy="0.0491285" iyz="-8.0419E-06" izz="0.0472376"/>	</inertial>
 </link>
 <link name = "world"/>
@@ -44,7 +43,7 @@
       <axis xyz="0 0 1" />
       <limit effort="0" lower="-2.965" upper="2.965" velocity="7.85" />
-</joint>
-<!-- Part 2 -->
-<link name ="${prefix}link_1">
+      <dynamics damping="1.0" friction="1.0"/>
+</joint>
+ <link name ="${prefix}link_1">
 	<collision>
 	<geometry>
@@ -60,8 +59,9 @@
 	</visual>
 	<inertial>
-		<origin xyz = "0.0 0.0 0.081" rpy = "0 0 0" />
-		<mass value = "4.85331"/>
-		<inertia ixx ="0.000533781" iyy=".055445798" izz=".02302818052" ixy="0.00012915752" ixz ="-0.002807595" iyz = "-0.000094967"/>
-	</inertial>
+        <origin xyz="-0.000010 -0.054550 0.028725" rpy="0 0 0"/>
+		<mass value = "2.13"/>
+        <inertia
+          ixx="${600 * 0.000048}" ixy="0.0" ixz="${600 * -0.000006}"
+          iyy="${600 * 0.000035}" iyz="0.0" izz="${600 * 0.000037}"/>	</inertial>
 </link>
 <gazebo reference= "${prefix}link_1" >
@@ -74,4 +74,5 @@
       <axis xyz="0 1 0" />
       <limit effort="0" lower="-1.745329" upper="2.530727" velocity="6.63" />
+      <dynamics damping="1.0" friction="1.0"/>
 </joint>
 <!--Part3-->
@@ -80,18 +81,20 @@
 		<origin xyz="0 0 0" rpy="0 0 0"/>
 		<geometry>
-			<mesh filename="package://fanuc_lrmate200id_support/meshes/lrmate200id/collision/link_2.stl"/>
-		</geometry>
-	</collision>
-	<visual>
-		<origin xyz="0 0 0" rpy="0 0 0"/>
-		<geometry>
-			<mesh filename = "package://fanuc_lrmate200id_support/meshes/lrmate200id/visual/link_2.stl"/>
-		</geometry>
-	</visual>
-	<inertial>
-		<origin xyz = "0 -0.00155 0.17556" rpy ="0 0 0"/>
-		<mass value = "7.96646"/>
-		<inertia ixx ="0.44125720672" iyy=".42103008445" izz=".03658588308" ixy="0.000023323" ixz ="-0.01624821395" iyz = "-0.00127983617"/>
-	</inertial>
+			<mesh filename="package://fanuc_lrmate200id_support/meshes/lrmate200id/collision/link_2.stl" />
+		</geometry>
+	</collision>
+	<visual>
+		<origin xyz="0 0 0" rpy="0 0 0"/>
+		<geometry>
+			<mesh filename = "package://fanuc_lrmate200id_support/meshes/lrmate200id/visual/link_2.stl" />
+		</geometry>
+	</visual>
+	<inertial>
+        <origin xyz="-0.002701 -0.000977 0.159466" rpy="0 0 0"/>
+		<mass value = "7.65"/>
+        <inertia
+          ixx="${600 * 0.000182}" ixy="0.0" ixz="0.0"
+          iyy="${600 * 0.000157}" iyz="${600 * -0.000001}"
+          izz="${600 * 0.000049}"/>	</inertial>
 </link>
 <gazebo reference= "${prefix}link_2" >
@@ -104,4 +107,5 @@
       <axis xyz="0 -1 0" />
       <limit effort="0" lower="-2.450966" upper="4.886922" velocity="9.08" />
+      <dynamics damping="1.0" friction="1.0"/>
 </joint>
 <link name="${prefix}link_3">
@@ -119,8 +123,10 @@
 	</visual>
 	<inertial>
-		<origin xyz = "0.008 0.00068 0.0177" rpy ="0 0 0"/>
-		<mass value = "2.401"/>
-		<inertia ixx ="0.00709493364" iyy=".08303386" izz=".007482747" ixy="0.000062924" ixz ="0.000131383" iyz = "0.000095227"/>
-	</inertial>
+        <origin xyz="-0.000065 0.017074 0.008866" rpy="0 0 0"/>
+		<mass value = "2.91"/>
+        <inertia
+          ixx="${600 * 0.000007}" ixy="0.0" ixz="${600 * -0.000001}"
+          iyy="${600 * 0.000008}" iyz="0.0"
+          izz="${600 * 0.000008}"/>	</inertial>
 </link>
 <gazebo reference= "${prefix}link_3" >
@@ -133,4 +139,5 @@
       <axis xyz="-1 0 0"/>
       <limit effort="0" lower="-3.315" upper="3.315" velocity="9.60" />
+      <dynamics damping="1.0" friction="1.0"/>
 </joint>
 <link name="${prefix}link_4">
@@ -138,5 +145,5 @@
 		<origin xyz ="0 0 0" rpy = "0 0 0" />
 		<geometry>
-			<mesh filename="package://fanuc_lrmate200id_support/meshes/lrmate200id/collision/link_4.stl"/>
+			<mesh filename="package://fanuc_lrmate200id_support/meshes/lrmate200id/collision/link_4.stl" />
 		</geometry>
 	</collision>
@@ -148,8 +155,10 @@
 	</visual>
 	<inertial>
-		<origin xyz = "0.24013 0 0" rpy ="0 0 0"/>
-		<mass value = "2.89084"/>
-		<inertia ixx ="0.004863267" iyy=".19336297539" izz=".19385148073" ixy="0.00303203667" ixz ="0.000018846079" iyz = "-0.00000096841"/>
-	</inertial>
+        <origin xyz="0.000067 0.002203 0.221634" rpy="0 0 0"/>
+		<mass value = "3.70"/>
+        <inertia
+          ixx="${600 * 0.000005}" ixy="0.0" ixz="0.0"
+          iyy="${600 * 0.000019}" iyz="0.0"
+          izz="${600 * 0.000019}"/>	</inertial>
 </link>
 <gazebo reference= "${prefix}link_4" >
@@ -162,4 +171,5 @@
       <axis xyz="0 -1 0"/>
       <limit effort="0" lower="-2.18" upper="2.18" velocity="9.51" />
+	  <dynamics damping="1.0" friction="1.0"/>
 </joint>
 <link name="${prefix}link_5">
@@ -177,8 +187,9 @@
 	</visual>
 	<inertial>
-		<origin xyz = "0.01573 0.003 -0.00006" rpy ="0 0 0"/>
-		<mass value = "0.043284"/>
-		<inertia ixx ="0.00029985018" iyy=".000661879" izz=".00064231094" ixy="-0.00000439197" ixz ="-0.000000345" iyz = "-0.00000008651"/>
-	</inertial>
+        <origin xyz="-0.000010 -0.054550 0.028725" rpy="0 0 0"/>
+		<mass value = "1.70"/>
+        <inertia
+          ixx="${600 * 0.00004}" ixy="0.0" ixz="${600 * -0.000004}"
+          iyy="${600 * 0.00003}" iyz="0.0" izz="${600 * 0.00003}"/>	</inertial>
 </link>
 <gazebo reference= "${prefix}link_5" >
@@ -191,4 +202,5 @@
       <axis xyz="-1 0 0"/>
       <limit effort="0" lower="-6.285" upper="6.285" velocity="17.45" />
+	  <dynamics damping="1.0" friction="1.0"/>
 </joint>
 <link name="${prefix}link_6">
@@ -206,7 +218,10 @@
 	</visual>
 	<inertial>
-		<origin xyz = "0.01573 0.003 -0.00006" rpy ="0 0 0"/>
-		<mass value = "0.043284"/>
-		<inertia ixx ="0.00029985018" iyy=".000661879" izz=".00064231094" ixy="-0.00000439197" ixz ="-0.000000345" iyz = "-0.00000008651"/>
+        <origin xyz="-0.000000 0.000000 -0.003006" rpy="0 0 0" />
+		<mass value = "0.137"/>
+        <inertia
+          ixx="0.01" ixy="0.0" ixz="0.0"
+          iyy="0.01" iyz="0.0"
+          izz="0.01"/>
 	</inertial>
 </link>
