Commit message: add gripper

File: fanuc_lrmate200id_gazebo/urdf/lrmate200id7l_gazebo.xacro (robot description, xacro)
@@ -1,5 +1,11 @@
-<?xml version="1.0"?>
+<?xml version="1.0" ?>
+<!-- =================================================================================== -->
+<!-- |    This document was autogenerated by xacro from /home/atas/catkin_ws/src/ROS_FANUC_LRMATE200ID/fanuc_experimental/fanuc_lrmate200id_support/urdf/lrmate200id7l.xacro | -->
+<!-- |    EDITING THIS FILE BY HAND IS NOT RECOMMENDED                                 | -->
+<!-- =================================================================================== -->
 <robot name="fanuc_lrmate200id7l" xmlns:xacro="http://www.ros.org/wiki/xacro">
-  <xacro:include filename="$(find fanuc_lrmate200id_gazebo)/urdf/lrmate200id7l_gazebo_macro.xacro"/>
-  <xacro:fanuc_lrmate200id7l prefix=""/>
+<xacro:include filename="$(find fanuc_lrmate200id_gazebo)/urdf/lrmate200id7l_gazebo_macro.xacro"/>
+<xacro:include filename="$(find fanuc_lrmate200id_gazebo)/urdf/gripper_macro.xacro"/>
+<xacro:fanuc_lrmate200id7l prefix=""/>
+<xacro:gripper prefix=""/>
 </robot>

File: fanuc_lrmate200id_gazebo/urdf/lrmate200id7l_gazebo_macro.xacro (robot description, xacro)
@@ -81,11 +81,11 @@
 		<origin xyz="0 0 0" rpy="0 0 0"/>
 		<geometry>
-			<mesh filename="package://fanuc_lrmate200id_support/meshes/lrmate200id7l/collision/link_2.stl" scale="0.001 0.001 0.001"/>
-		</geometry>
-	</collision>
-	<visual>
-		<origin xyz="0 0 0" rpy="0 0 0"/>
-		<geometry>
-			<mesh filename = "package://fanuc_lrmate200id_support/meshes/lrmate200id7l/visual/link_2.stl" scale="0.001 0.001 0.001"/>
+			<mesh filename="package://fanuc_lrmate200id_support/meshes/lrmate200id7l/collision/link_2.stl" scale ="0.001 0.001 0.001"  />
+		</geometry>
+	</collision>
+	<visual>
+		<origin xyz="0 0 0" rpy="0 0 0"/>
+		<geometry>
+			<mesh filename = "package://fanuc_lrmate200id_support/meshes/lrmate200id7l/visual/link_2.stl"  scale ="0.001 0.001 0.001"/>
 		</geometry>
 	</visual>
@@ -145,5 +145,5 @@
 		<origin xyz ="0 0 0" rpy = "0 0 0" />
 		<geometry>
-			<mesh filename="package://fanuc_lrmate200id_support/meshes/lrmate200id7l/collision/link_4.stl" scale="0.001 0.001 0.001"/>
+			<mesh filename="package://fanuc_lrmate200id_support/meshes/lrmate200id7l/collision/link_4.stl"  scale ="0.001 0.001 0.001"/>
 		</geometry>
 	</collision>
@@ -151,5 +151,5 @@
 		<origin xyz ="0 0 0" rpy = "0 0 0" />
 		<geometry>
-			<mesh filename="package://fanuc_lrmate200id_support/meshes/lrmate200id7l/visual/link_4.stl" scale="0.001 0.001 0.001"/>
+			<mesh filename="package://fanuc_lrmate200id_support/meshes/lrmate200id7l/visual/link_4.stl" scale ="0.001 0.001 0.001"/>
 		</geometry>
 	</visual>

File: fanuc_lrmate200id_support/urdf/lrmate200id7l.xacro (robot description, xacro)
@@ -1,5 +1,7 @@
 <?xml version="1.0"?>
-<robot name="fanuc_lrmate200id7l" xmlns:xacro="http://wiki.ros.org/xacro">
+<robot name="fanuc_lrmate200id7l" xmlns:xacro="http://www.ros.org/wiki/xacro">
   <xacro:include filename="$(find fanuc_lrmate200id_support)/urdf/lrmate200id7l_macro.xacro"/>
+  <xacro:include filename="$(find fanuc_lrmate200id_support)/urdf/gripper_macro.xacro" />
   <xacro:fanuc_lrmate200id7l prefix=""/>
+  <xacro:gripper prefix=""/>
 </robot>

File: fanuc_lrmate200id_support/urdf/lrmate200id7l_macro.xacro (robot description, xacro)
@@ -1,4 +1,4 @@
 <?xml version="1.0"?>
-<robot xmlns:xacro="http://wiki.ros.org/xacro">
+<robot xmlns:xacro="http://www.ros.org/wiki/xacro">
   <xacro:include filename="$(find fanuc_resources)/urdf/common_materials.xacro"/>
   <xacro:macro name="fanuc_lrmate200id7l" params="prefix">
@@ -166,6 +166,19 @@
       <child link="${prefix}flange" />
     </joint>
-    <!-- ROS-Industrial 'tool0' frame: all-zeros tool frame -->
-    <link name="${prefix}tool0" />
+    <link name="${prefix}tool0">
+      <visual>
+        <origin xyz="0 0 0" rpy="0 0 0"/>
+        <geometry>
+          <mesh filename="package://fanuc_lrmate200id_support/meshes/lrmate200id/visual/link_6.stl"/>
+        </geometry>
+        <xacro:material_fanuc_black />
+      </visual>
+      <collision>
+        <origin xyz="0 0 0" rpy="0 0 0"/>
+        <geometry>
+          <mesh filename="package://fanuc_lrmate200id_support/meshes/lrmate200id/collision/link_6.stl"/>
+        </geometry>
+      </collision>
+    </link>
     <joint name="${prefix}link_6-tool0" type="fixed">
       <origin xyz="0 0 0" rpy="${pi} ${-pi/2.0} 0" />
