Commit message: add gripper control

File: fanuc_lrmate200id_gazebo/urdf/gripper_macro.xacro (robot description, xacro)
@@ -9,5 +9,5 @@
         <axis xyz="0 0 1" />
         <dynamics damping="0.7" />
-        <limit effort="100" lower="-0.5232" upper="0.5232" velocity="100" />
+        <limit effort="100" lower="0" upper="0" velocity="100" />
     </joint>
     <!-- Gripper Base -->
@@ -44,5 +44,5 @@
         <axis xyz="0 1 0" />
         <dynamics damping="0.7" />
-        <limit effort="1" lower="-0.0872" upper="0.0872" velocity="6.1087" />
+        <limit effort="1" lower="-0.4" upper="0.4" velocity="6.1087" />
     </joint>
     <!-- Finger 3-->
@@ -77,5 +77,5 @@
         <axis xyz="0 1 0" />
         <dynamics damping="0.7" />
-        <limit effort="1" lower="-0.0872" upper="0.0872" velocity="6.1087" />
+        <limit effort="1" lower="-0.4" upper="0.4" velocity="6.1087" />
     </joint>
     <!-- Finger 1-->
@@ -109,5 +109,5 @@
         <axis xyz="0 1 0" />
         <dynamics damping="0.7" />
-        <limit effort="1" lower="-0.0872" upper="0.0872" velocity="6.1087" />
+        <limit effort="1" lower="-0.4" upper="0.4" velocity="6.1087" />
     </joint>
     <!-- Finger 2-->
@@ -137,8 +137,8 @@
         <type>transmission_interface/SimpleTransmission</type>
         <joint name="Part6_Gripper_Base">
-            <hardwareInterface>hardware_interface/PositionJointInterface</hardwareInterface>
+            <hardwareInterface>hardware_interface/EffortJointInterface</hardwareInterface>
         </joint>
         <actuator name="Part6_Gripper_Base_motor">
-            <hardwareInterface>hardware_interface/PositionJointInterface</hardwareInterface>
+            <hardwareInterface>hardware_interface/EffortJointInterface</hardwareInterface>
             <mechanicalReduction>1</mechanicalReduction>
         </actuator>
@@ -147,8 +147,8 @@
         <type>transmission_interface/SimpleTransmission</type>
         <joint name="Gripper_Finger3">
-            <hardwareInterface>hardware_interface/PositionJointInterface</hardwareInterface>
+            <hardwareInterface>hardware_interface/EffortJointInterface</hardwareInterface>
         </joint>
         <actuator name="Gripper_Finger3_motor">
-            <hardwareInterface>hardware_interface/PositionJointInterface</hardwareInterface>
+            <hardwareInterface>hardware_interface/EffortJointInterface</hardwareInterface>
             <mechanicalReduction>1</mechanicalReduction>
         </actuator>
@@ -157,8 +157,8 @@
         <type>transmission_interface/SimpleTransmission</type>
         <joint name="Gripper_Finger1">
-            <hardwareInterface>hardware_interface/PositionJointInterface</hardwareInterface>
+            <hardwareInterface>hardware_interface/EffortJointInterface</hardwareInterface>
         </joint>
         <actuator name="Gripper_Finger1_motor">
-            <hardwareInterface>hardware_interface/PositionJointInterface</hardwareInterface>
+            <hardwareInterface>hardware_interface/EffortJointInterface</hardwareInterface>
             <mechanicalReduction>1</mechanicalReduction>
         </actuator>
@@ -167,8 +167,8 @@
         <type>transmission_interface/SimpleTransmission</type>
         <joint name="Gripper_Finger2">
-            <hardwareInterface>hardware_interface/PositionJointInterface</hardwareInterface>
+            <hardwareInterface>hardware_interface/EffortJointInterface</hardwareInterface>
         </joint>
         <actuator name="Gripper_Finger2_motor">
-            <hardwareInterface>hardware_interface/PositionJointInterface</hardwareInterface>
+            <hardwareInterface>hardware_interface/EffortJointInterface</hardwareInterface>
             <mechanicalReduction>1</mechanicalReduction>
         </actuator>

Commit message: Add workcell simulation

File: fanuc_lrmate200id_gazebo/urdf/gripper_macro.xacro (robot description, xacro)
@@ -8,5 +8,5 @@
         <origin rpy="0 -1.57 0" xyz="0 0 0" />
         <axis xyz="0 0 1" />
-        <dynamics damping="0.7" />
+        <dynamics damping="5" friction="1.2"/>
         <limit effort="100" lower="0" upper="0" velocity="100" />
     </joint>
@@ -30,5 +30,5 @@
 <inertial>
             <origin rpy="0 0 0" xyz="0.00112 0.04196 0" />
-            <mass value="1.067" />
+            <mass value="0.1" />
             <inertia ixx="0.00372062398" ixy="-0.000013337910" ixz="0.000000013" iyy=".00223540544" iyz="-0.00000003496" izz=".003641916" />
         </inertial>
@@ -43,5 +43,5 @@
         <origin rpy="0 0 0" xyz="0.04448 0 -0.09533" />
         <axis xyz="0 1 0" />
-        <dynamics damping="0.7" />
+        <dynamics damping="5" friction="1.2"/>
         <limit effort="1" lower="-0.4" upper="0.4" velocity="6.1087" />
     </joint>
@@ -76,5 +76,5 @@
         <origin rpy="0 0 0" xyz="-0.04448 0.04 -0.09533" />
         <axis xyz="0 1 0" />
-        <dynamics damping="0.7" />
+        <dynamics damping="5" friction="1.2"/>
         <limit effort="1" lower="-0.4" upper="0.4" velocity="6.1087" />
     </joint>
@@ -108,5 +108,5 @@
         <origin rpy="0 0 0" xyz="-0.04448 -0.04 -0.09533" />
         <axis xyz="0 1 0" />
-        <dynamics damping="0.7" />
+        <dynamics damping="5" friction="1.2"/>
         <limit effort="1" lower="-0.4" upper="0.4" velocity="6.1087" />
     </joint>
@@ -134,11 +134,44 @@
         </inertial>
     </link>
+      <gazebo reference="Gripper_Finger1">
+    <implicitSpringDamper>1</implicitSpringDamper>
+      </gazebo>
+      <gazebo reference="Gripper_Finger2">
+    <implicitSpringDamper>1</implicitSpringDamper>
+      </gazebo>
+      <gazebo reference="Gripper_Finger3">
+    <implicitSpringDamper>1</implicitSpringDamper>
+      </gazebo>
+    <gazebo reference="Finger1">
+  <kp>1000000.0</kp>
+  <kd>1.0</kd>
+  <mu1>0.8</mu1>
+  <mu2>0.8</mu2>
+  <maxVel>0.0</maxVel>
+  <minDepth>0.001</minDepth>
+    </gazebo>
+    <gazebo reference="Finger2">
+  <kp>1000000.0</kp>
+  <kd>1.0</kd>
+  <mu1>0.8</mu1>
+  <mu2>0.8</mu2>
+  <maxVel>0.0</maxVel>
+  <minDepth>0.001</minDepth>
+    </gazebo>
+    <gazebo reference="Finger3">
+  <kp>1000000.0</kp>
+  <kd>1.0</kd>
+  <mu1>0.8</mu1>
+  <mu2>0.8</mu2>
+  <maxVel>0.0</maxVel>
+  <minDepth>0.001</minDepth>
+    </gazebo>
     <transmission name="trans_Part6_Gripper_Base">
         <type>transmission_interface/SimpleTransmission</type>
         <joint name="Part6_Gripper_Base">
-            <hardwareInterface>hardware_interface/EffortJointInterface</hardwareInterface>
+            <hardwareInterface>hardware_interface/PositionJointInterface</hardwareInterface>
         </joint>
         <actuator name="Part6_Gripper_Base_motor">
-            <hardwareInterface>hardware_interface/EffortJointInterface</hardwareInterface>
+            <hardwareInterface>hardware_interface/PositionJointInterface</hardwareInterface>
             <mechanicalReduction>1</mechanicalReduction>
         </actuator>
@@ -147,8 +180,8 @@
         <type>transmission_interface/SimpleTransmission</type>
         <joint name="Gripper_Finger3">
-            <hardwareInterface>hardware_interface/EffortJointInterface</hardwareInterface>
+            <hardwareInterface>hardware_interface/PositionJointInterface</hardwareInterface>
         </joint>
         <actuator name="Gripper_Finger3_motor">
-            <hardwareInterface>hardware_interface/EffortJointInterface</hardwareInterface>
+            <hardwareInterface>hardware_interface/PositionJointInterface</hardwareInterface>
             <mechanicalReduction>1</mechanicalReduction>
         </actuator>
@@ -157,8 +190,8 @@
         <type>transmission_interface/SimpleTransmission</type>
         <joint name="Gripper_Finger1">
-            <hardwareInterface>hardware_interface/EffortJointInterface</hardwareInterface>
+            <hardwareInterface>hardware_interface/PositionJointInterface</hardwareInterface>
         </joint>
         <actuator name="Gripper_Finger1_motor">
-            <hardwareInterface>hardware_interface/EffortJointInterface</hardwareInterface>
+            <hardwareInterface>hardware_interface/PositionJointInterface</hardwareInterface>
             <mechanicalReduction>1</mechanicalReduction>
         </actuator>
@@ -167,8 +200,8 @@
         <type>transmission_interface/SimpleTransmission</type>
         <joint name="Gripper_Finger2">
-            <hardwareInterface>hardware_interface/EffortJointInterface</hardwareInterface>
+            <hardwareInterface>hardware_interface/PositionJointInterface</hardwareInterface>
         </joint>
         <actuator name="Gripper_Finger2_motor">
-            <hardwareInterface>hardware_interface/EffortJointInterface</hardwareInterface>
+            <hardwareInterface>hardware_interface/PositionJointInterface</hardwareInterface>
             <mechanicalReduction>1</mechanicalReduction>
         </actuator>

File: fanuc_lrmate200id_gazebo/urdf/lrmate200id7l_gazebo_macro.xacro (robot description, xacro)
@@ -43,5 +43,5 @@
       <axis xyz="0 0 1" />
       <limit effort="0" lower="-2.965" upper="2.965" velocity="7.85" />
-      <dynamics damping="1.0" friction="1.0"/>
+      <dynamics damping="1.0" friction="5.0"/>
 </joint>
  <link name ="${prefix}link_1">
@@ -60,5 +60,5 @@
 	<inertial>
         <origin xyz="-0.000010 -0.054550 0.028725" rpy="0 0 0"/>
-		<mass value = "2.13"/>
+		<mass value = "1"/>
         <inertia
           ixx="${600 * 0.000048}" ixy="0.0" ixz="${600 * -0.000006}"
@@ -74,5 +74,5 @@
       <axis xyz="0 1 0" />
       <limit effort="0" lower="-1.745329" upper="2.530727" velocity="6.63" />
-      <dynamics damping="1.0" friction="1.0"/>
+      <dynamics damping="1.0" friction="5.0"/>
 </joint>
 <!--Part3-->
@@ -92,5 +92,5 @@
 	<inertial>
         <origin xyz="-0.002701 -0.000977 0.159466" rpy="0 0 0"/>
-		<mass value = "7.65"/>
+		<mass value = "1"/>
         <inertia
           ixx="${600 * 0.000182}" ixy="0.0" ixz="0.0"
@@ -107,5 +107,5 @@
       <axis xyz="0 -1 0" />
       <limit effort="0" lower="-2.450966" upper="4.886922" velocity="9.08" />
-      <dynamics damping="1.0" friction="1.0"/>
+      <dynamics damping="1.0" friction="5.0"/>
 </joint>
 <link name="${prefix}link_3">
@@ -124,5 +124,5 @@
 	<inertial>
         <origin xyz="-0.000065 0.017074 0.008866" rpy="0 0 0"/>
-		<mass value = "2.91"/>
+		<mass value = "1"/>
         <inertia
           ixx="${600 * 0.000007}" ixy="0.0" ixz="${600 * -0.000001}"
@@ -139,5 +139,5 @@
       <axis xyz="-1 0 0"/>
       <limit effort="0" lower="-3.315" upper="3.315" velocity="9.60" />
-      <dynamics damping="1.0" friction="1.0"/>
+      <dynamics damping="1.0" friction="5.0"/>
 </joint>
 <link name="${prefix}link_4">
@@ -156,5 +156,5 @@
 	<inertial>
         <origin xyz="0.000067 0.002203 0.221634" rpy="0 0 0"/>
-		<mass value = "3.70"/>
+		<mass value = "1"/>
         <inertia
           ixx="${600 * 0.000005}" ixy="0.0" ixz="0.0"
@@ -171,5 +171,5 @@
       <axis xyz="0 -1 0"/>
       <limit effort="0" lower="-2.18" upper="2.18" velocity="9.51" />
-	  <dynamics damping="1.0" friction="1.0"/>
+	  <dynamics damping="1.0" friction="5.0"/>
 </joint>
 <link name="${prefix}link_5">
@@ -188,5 +188,5 @@
 	<inertial>
         <origin xyz="-0.000010 -0.054550 0.028725" rpy="0 0 0"/>
-		<mass value = "1.70"/>
+		<mass value = "1"/>
         <inertia
           ixx="${600 * 0.00004}" ixy="0.0" ixz="${600 * -0.000004}"
@@ -202,5 +202,5 @@
       <axis xyz="-1 0 0"/>
       <limit effort="0" lower="-6.285" upper="6.285" velocity="17.45" />
-	  <dynamics damping="1.0" friction="1.0"/>
+	  <dynamics damping="1.0" friction="5.0"/>
 </joint>
 <link name="${prefix}link_6">

Commit message: add .dae file to avoid gazebo load error

File: fanuc_lrmate200id_gazebo/urdf/gripper_macro.xacro (robot description, xacro)
@@ -16,5 +16,5 @@
             <origin rpy="-1.57 0 0" xyz="-0.065 -0.065 0" />
             <geometry>
-                <mesh filename="package://fanuc_lrmate200id_support/meshes/gripper/collision/Gripper_base.STL" scale="0.001 0.001 0.001" />
+                <mesh filename="package://fanuc_lrmate200id_support/meshes/gripper/collision/Gripper_base.dae" scale="0.001 0.001 0.001" />
             </geometry>
         </collision>
@@ -22,5 +22,5 @@
             <origin rpy="-1.57 0 0" xyz="-0.065 -0.065 0" />
             <geometry>
-                <mesh filename="package://fanuc_lrmate200id_support/meshes/gripper/visual/Gripper_base.STL" scale="0.001 0.001 0.001" />
+                <mesh filename="package://fanuc_lrmate200id_support/meshes/gripper/visual/Gripper_base.dae" scale="0.001 0.001 0.001" />
             </geometry>
             <material name="">
@@ -51,5 +51,5 @@
             <origin rpy="-1.57 0 3.14" xyz="0.075 0.038 0.075" />
             <geometry>
-                <mesh filename="package://fanuc_lrmate200id_support/meshes/gripper/collision/Gripper_finger.STL" scale="0.001 0.001 0.001" />
+                <mesh filename="package://fanuc_lrmate200id_support/meshes/gripper/collision/Gripper_finger.dae" scale="0.001 0.001 0.001" />
             </geometry>
         </collision>
@@ -57,5 +57,5 @@
             <origin rpy="-1.57 0 3.14" xyz="0.075 0.038 0.075" />
             <geometry>
-                <mesh filename="package://fanuc_lrmate200id_support/meshes/gripper/visual/Gripper_finger.STL" scale="0.001 0.001 0.001" />
+                <mesh filename="package://fanuc_lrmate200id_support/meshes/gripper/visual/Gripper_finger.dae" scale="0.001 0.001 0.001" />
             </geometry>
             <material name="">
@@ -84,11 +84,11 @@
             <origin rpy="-1.57 0 0" xyz="-0.075 -0.038 0.075" />
             <geometry>
-                <mesh filename="package://fanuc_lrmate200id_support/meshes/gripper/collision/Gripper_finger.STL" scale="0.001 0.001 0.001" />
-            </geometry>
-        </collision>
-        <visual>
-            <origin rpy="-1.57 0 0" xyz="-0.075 -0.038 0.075" />
-            <geometry>
-                <mesh filename="package://fanuc_lrmate200id_support/meshes/gripper/visual/Gripper_finger.STL" scale="0.001 0.001 0.001" />
+                <mesh filename="package://fanuc_lrmate200id_support/meshes/gripper/collision/Gripper_finger.dae" scale="0.001 0.001 0.001" />
+            </geometry>
+        </collision>
+        <visual>
+            <origin rpy="-1.57 0 0" xyz="-0.075 -0.038 0.075" />
+            <geometry>
+                <mesh filename="package://fanuc_lrmate200id_support/meshes/gripper/visual/Gripper_finger.dae" scale="0.001 0.001 0.001" />
             </geometry>
             <material name="">
@@ -116,11 +116,11 @@
             <origin rpy="-1.57 0 0" xyz="-0.075 -0.038 0.075" />
             <geometry>
-                <mesh filename="package://fanuc_lrmate200id_support/meshes/gripper/collision/Gripper_finger.STL" scale="0.001 0.001 0.001" />
-            </geometry>
-        </collision>
-        <visual>
-            <origin rpy="-1.57 0 0" xyz="-0.075 -0.038 0.075" />
-            <geometry>
-                <mesh filename="package://fanuc_lrmate200id_support/meshes/gripper/visual/Gripper_finger.STL" scale="0.001 0.001 0.001" />
+                <mesh filename="package://fanuc_lrmate200id_support/meshes/gripper/collision/Gripper_finger.dae" scale="0.001 0.001 0.001" />
+            </geometry>
+        </collision>
+        <visual>
+            <origin rpy="-1.57 0 0" xyz="-0.075 -0.038 0.075" />
+            <geometry>
+                <mesh filename="package://fanuc_lrmate200id_support/meshes/gripper/visual/Gripper_finger.dae" scale="0.001 0.001 0.001" />
             </geometry>
             <material name="">
