Commit message: Random Movement for object

File: fanuc_lrmate200id_gazebo/urdf/asus_xtion_macro.xacro (robot description, xacro)
@@ -6,5 +6,5 @@
     <parent link="base_link" />
     <child link="camera_link" />
-    <origin rpy="0 1.57 0" xyz="0.6 -0.3 0.8" />
+    <origin rpy="0 1.57 0" xyz="0.6 -0.3 1.4" />
     <axis xyz="0 0 0" />
 </joint>

File: fanuc_lrmate200id_gazebo/urdf/lrmate200id7l_gazebo_macro.xacro (robot description, xacro)
@@ -32,5 +32,5 @@
 	<parent link="world"/>
 	<child link="${prefix}base_link" />
-	<origin xyz = "0 0 0" rpy = "0 0 0"/>
+	<origin xyz = "0.7 -1.6 0.7" rpy = "0 0 0"/>
 </joint>
 <gazebo reference= "${prefix}base_link" >

Commit message: add dummy link to xtion

File: fanuc_lrmate200id_gazebo/urdf/asus_xtion_macro.xacro (robot description, xacro)
@@ -9,4 +9,18 @@
     <axis xyz="0 0 0" />
 </joint>
+<joint name="dummy_joint" type="fixed">
+    <parent link="camera_link" />
+    <child link="dummy_link" />
+    <origin rpy="0 1.57 0" xyz=" 0 0 0" />
+    <axis xyz="0 0 0" />
+</joint>
+<link name="dummy_link"/>
+<joint name="dope_joint" type="fixed">
+    <parent link="dummy_link" />
+    <child link="dope_link" />
+    <origin rpy="0 0 -1.57" xyz=" 0 0 0" />
+    <axis xyz="0 0 0" />
+</joint>
+<link name="dope_link"/>
 <link name="camera_link">
     <collision name="collision">

Commit message: camera postion adjustment

File: fanuc_lrmate200id_gazebo/urdf/asus_xtion_macro.xacro (robot description, xacro)
@@ -6,5 +6,5 @@
     <parent link="base_link" />
     <child link="camera_link" />
-    <origin rpy="0 1.57 0" xyz="0.6 -0.3 1.4" />
+    <origin rpy="0 1.57 0" xyz="0.6 -0.3 1.1" />
     <axis xyz="0 0 0" />
 </joint>

Commit message: change height of camera

File: fanuc_lrmate200id_gazebo/urdf/asus_xtion_macro.xacro (robot description, xacro)
@@ -6,5 +6,5 @@
     <parent link="base_link" />
     <child link="camera_link" />
-    <origin rpy="0 1.57 0" xyz="0.6 -0.3 1.1" />
+    <origin rpy="0 1.57 0" xyz="0.6 -0.3 1.3" />
     <axis xyz="0 0 0" />
 </joint>

Commit message: pcd dataset changes

File: fanuc_lrmate200id_gazebo/urdf/asus_xtion_macro.xacro (robot description, xacro)
@@ -6,5 +6,5 @@
     <parent link="base_link" />
     <child link="camera_link" />
-    <origin rpy="0 1.57 0" xyz="0.6 -0.3 1.3" />
+    <origin rpy="0 1.57 0" xyz="0.6 -0.7 1.1" />
     <axis xyz="0 0 0" />
 </joint>
@@ -52,6 +52,6 @@
           </image>
           <clip>
-            <near>0.3</near>
-            <far>3.5</far>
+            <near>0.2</near>
+            <far>0.8</far>
           </clip>
         </camera>
@@ -69,6 +69,6 @@
           <pointCloudTopicName>/camera/depth/points</pointCloudTopicName>
           <frameName>camera_link</frameName>
-          <pointCloudCutoff>0.5</pointCloudCutoff>
-          <pointCloudCutoffMax>3.0</pointCloudCutoffMax>
+          <pointCloudCutoff>0.2</pointCloudCutoff>
+          <pointCloudCutoffMax>0.8</pointCloudCutoffMax>
           <distortionK1>0</distortionK1>
           <distortionK2>0</distortionK2>

Commit message: point_cloud_dataset_branch

File: fanuc_lrmate200id_gazebo/urdf/asus_xtion_macro.xacro (robot description, xacro)
@@ -6,5 +6,5 @@
     <parent link="base_link" />
     <child link="camera_link" />
-    <origin rpy="0 1.57 0" xyz="0.6 -0.7 1.1" />
+    <origin rpy="0 1.57 0" xyz="0.6 -0.9 1.6" />
     <axis xyz="0 0 0" />
 </joint>
@@ -53,5 +53,5 @@
           <clip>
             <near>0.2</near>
-            <far>0.8</far>
+            <far>3.0</far>
           </clip>
         </camera>
@@ -70,5 +70,5 @@
           <frameName>camera_link</frameName>
           <pointCloudCutoff>0.2</pointCloudCutoff>
-          <pointCloudCutoffMax>0.8</pointCloudCutoffMax>
+          <pointCloudCutoffMax>1.2</pointCloudCutoffMax>
           <distortionK1>0</distortionK1>
           <distortionK2>0</distortionK2>

Commit message: fix simulator issues

File: fanuc_lrmate200id_gazebo/urdf/asus_xtion_macro.xacro (robot description, xacro)
@@ -6,21 +6,7 @@
     <parent link="base_link" />
     <child link="camera_link" />
-    <origin rpy="0 1.57 0" xyz="0.6 -0.9 1.6" />
+    <origin rpy="0 1.57 0" xyz="0.6 0.0 1.6" />
     <axis xyz="0 0 0" />
 </joint>
-<joint name="dummy_joint" type="fixed">
-    <parent link="camera_link" />
-    <child link="dummy_link" />
-    <origin rpy="0 1.57 0" xyz=" 0 0 0" />
-    <axis xyz="0 0 0" />
-</joint>
-<link name="dummy_link"/>
-<joint name="dope_joint" type="fixed">
-    <parent link="dummy_link" />
-    <child link="dope_link" />
-    <origin rpy="0 0 -1.57" xyz=" 0 0 0" />
-    <axis xyz="0 0 0" />
-</joint>
-<link name="dope_link"/>
 <link name="camera_link">
     <collision name="collision">

File: fanuc_lrmate200id_gazebo/urdf/lrmate200id7l_gazebo_macro.xacro (robot description, xacro)
@@ -32,5 +32,5 @@
 	<parent link="world"/>
 	<child link="${prefix}base_link" />
-	<origin xyz = "0.7 -1.6 0.7" rpy = "0 0 0"/>
+	<origin xyz = "0.0 0.0 0.0" rpy = "0 0 0"/>
 </joint>
 <gazebo reference= "${prefix}base_link" >
