Commit message: add gazebo support

File: fanuc_lrmate200id_gazebo/urdf/lrmate200id7l.xacro (robot description, xacro)
@@ -5,9 +5,12 @@
 <!-- =================================================================================== -->
 <robot name="fanuc_lrmate200id7l" xmlns:xacro="http://www.ros.org/wiki/xacro">
-<xacro:include filename="$(find fanuc_lrmate200id_gazebo)/urdf/lrmate200id7l_gazebo_macro.xacro"/>
-<xacro:include filename="$(find fanuc_lrmate200id_gazebo)/urdf/gripper_macro.xacro"/>
-<xacro:include filename="$(find fanuc_lrmate200id_gazebo)/urdf/asus_xtion_macro.xacro"/>
-<xacro:fanuc_lrmate200id7l prefix=""/>
-<xacro:gripper prefix=""/>
-<xacro:asus_xtion prefix=""/>
+<xacro:include filename="$(find fanuc_lrmate200id_gazebo)/urdf/lrmate200id7l_macro.xacro"/>
+  <xacro:fanuc_lrmate200id7l_robot prefix=""/>
+  <!-- Fix robot to Gazebo world -->
+  <link name="world"/>
+  <joint name="world-base_link-fixed" type="fixed">
+    <parent link="world"/>
+    <child link="base_link"/>
+    <origin xyz="0.0 0.0 0.0" rpy="0.0 0.0 0.0" />
+  </joint>
 </robot>

File: fanuc_lrmate200id_support/urdf/lrmate200id7l.xacro (robot description, xacro)
@@ -3,12 +3,3 @@
   <xacro:include filename="$(find fanuc_lrmate200id_support)/urdf/lrmate200id7l_macro.xacro"/>
   <xacro:fanuc_lrmate200id7l prefix=""/>
-       <!-- Part 6 Gripper Base Joint -->
-<joint name="camera_joint" type="fixed">
-    <parent link="link_4" />
-    <child link="camera_link" />
-    <origin rpy="-0.0037 1.50600 -0.0031"
-     xyz="0.32273 0.01841 -0.06556" />
-    <axis xyz="0 0 0" />
-</joint>
-<link name="camera_link"/>
 </robot>

File: fanuc_lrmate200id_support/urdf/lrmate200id7l_macro.xacro (robot description, xacro)
@@ -18,4 +18,11 @@
         </geometry>
       </collision>
+      <inertial>
+          <mass value="10.733459"/>
+          <origin xyz="0.014288 0.000001 0.122264" rpy="0.0 0.0 0.0"/>
+          <inertia ixx="0.096590" ixy="-0.000005" ixz="-0.003803"
+                                  iyy="0.087591"  iyz="-0.000001"
+                                                  izz="0.081632"/>
+      </inertial>
     </link>
     <link name="${prefix}link_1">
@@ -33,4 +40,11 @@
         </geometry>
       </collision>
+      <inertial>
+          <mass value="16.934564"/>
+          <origin xyz="0.019143 0.024764 -0.064596" rpy="0.0 0.0 0.0"/>
+          <inertia ixx="0.222318" ixy="0.016499" ixz="0.023794"
+                                  iyy="0.208959" iyz="0.031663"
+                                                 izz="0.157081"/>
+      </inertial>
     </link>
     <link name="${prefix}link_2">
@@ -48,4 +62,11 @@
         </geometry>
       </collision>
+      <inertial>
+          <mass value="12.98711"/>
+          <origin xyz="-0.000008 0.221181 0.173052" rpy="0.0 0.0 0.0"/>
+          <inertia ixx="0.425299" ixy="0.000005" ixz="-0.000004"
+                                  iyy="0.452311" iyz="-0.002920"
+                                                 izz="0.054493"/>
+      </inertial>
     </link>
     <link name="${prefix}link_3">
@@ -63,4 +84,11 @@
         </geometry>
       </collision>
+      <inertial>
+          <mass value="7.50151"/>
+          <origin xyz="0.000002 0.065008 0.003572" rpy="0.0 0.0 0.0"/>
+          <inertia ixx="0.058902" ixy="0.000000" ixz="0.000001"
+                                  iyy="0.056884" iyz="-0.003672"
+                                                 izz="0.034271"/>
+      </inertial>
     </link>
     <link name="${prefix}link_4">
@@ -78,4 +106,11 @@
         </geometry>
       </collision>
+      <inertial>
+          <mass value="4.54015"/>
+          <origin xyz="-0.002488 0.049988 0.296156" rpy="0.0 0.0 0.0"/>
+          <inertia ixx="0.043246" ixy="0.000003" ixz="-0.000683"
+                                  iyy="0.038394" iyz="-0.000004"
+                                                 izz="0.014525"/>
+      </inertial>
     </link>
     <link name="${prefix}link_5">
@@ -93,4 +128,11 @@
         </geometry>
       </collision>
+      <inertial>
+          <mass value="0.56876"/>
+          <origin xyz="0.000000 0.049931 0.222823" rpy="0.0 0.0 0.0"/>
+          <inertia ixx="0.001084" ixy="0.000000" ixz="0.000000"
+                                  iyy="0.001123" iyz="0.000001"
+                                                 izz="0.000383"/>
+      </inertial>
     </link>
     <link name="${prefix}link_6">
@@ -108,4 +150,11 @@
         </geometry>
       </collision>
+      <inertial>
+          <mass value="0.03098"/>
+          <origin xyz="-0.000243 0.050000 -0.006293" rpy="0.0 0.0 0.0"/>
+          <inertia ixx="0.000012" ixy="0.000000" ixz="0.000000"
+                                  iyy="0.000011" iyz="0.000000"
+                                                 izz="0.000022"/>
+      </inertial>
     </link>
     <!-- joints: main serial chain -->

File: fanuc_lrmate200id_support/urdf/lrmate200id_macro.xacro (robot description, xacro)
@@ -18,4 +18,11 @@
         </geometry>
       </collision>
+      <inertial>
+          <mass value="10.733459"/>
+          <origin xyz="0.014288 0.000001 0.122264" rpy="0.0 0.0 0.0"/>
+          <inertia ixx="0.096590" ixy="-0.000005" ixz="-0.003803"
+                                  iyy="0.087591"  iyz="-0.000001"
+                                                  izz="0.081632"/>
+      </inertial>
     </link>
     <link name="${prefix}link_1">
@@ -33,4 +40,11 @@
         </geometry>
       </collision>
+      <inertial>
+          <mass value="16.934564"/>
+          <origin xyz="0.019143 0.024764 -0.064596" rpy="0.0 0.0 0.0"/>
+          <inertia ixx="0.222318" ixy="0.016499" ixz="0.023794"
+                                  iyy="0.208959" iyz="0.031663"
+                                                 izz="0.157081"/>
+      </inertial>
     </link>
     <link name="${prefix}link_2">
@@ -48,4 +62,11 @@
         </geometry>
       </collision>
+      <inertial>
+          <mass value="12.98711"/>
+          <origin xyz="-0.000008 0.221181 0.173052" rpy="0.0 0.0 0.0"/>
+          <inertia ixx="0.425299" ixy="0.000005" ixz="-0.000004"
+                                  iyy="0.452311" iyz="-0.002920"
+                                                 izz="0.054493"/>
+      </inertial>
     </link>
     <link name="${prefix}link_3">
@@ -63,4 +84,11 @@
         </geometry>
       </collision>
+      <inertial>
+          <mass value="7.50151"/>
+          <origin xyz="0.000002 0.065008 0.003572" rpy="0.0 0.0 0.0"/>
+          <inertia ixx="0.058902" ixy="0.000000" ixz="0.000001"
+                                  iyy="0.056884" iyz="-0.003672"
+                                                 izz="0.034271"/>
+      </inertial>
     </link>
     <link name="${prefix}link_4">
@@ -78,4 +106,11 @@
         </geometry>
       </collision>
+      <inertial>
+          <mass value="4.54015"/>
+          <origin xyz="-0.002488 0.049988 0.296156" rpy="0.0 0.0 0.0"/>
+          <inertia ixx="0.043246" ixy="0.000003" ixz="-0.000683"
+                                  iyy="0.038394" iyz="-0.000004"
+                                                 izz="0.014525"/>
+      </inertial>
     </link>
     <link name="${prefix}link_5">
@@ -93,4 +128,11 @@
         </geometry>
       </collision>
+      <inertial>
+          <mass value="0.56876"/>
+          <origin xyz="0.000000 0.049931 0.222823" rpy="0.0 0.0 0.0"/>
+          <inertia ixx="0.001084" ixy="0.000000" ixz="0.000000"
+                                  iyy="0.001123" iyz="0.000001"
+                                                 izz="0.000383"/>
+      </inertial>
     </link>
     <link name="${prefix}link_6">
@@ -108,4 +150,11 @@
         </geometry>
       </collision>
+      <inertial>
+          <mass value="0.03098"/>
+          <origin xyz="-0.000243 0.050000 -0.006293" rpy="0.0 0.0 0.0"/>
+          <inertia ixx="0.000012" ixy="0.000000" ixz="0.000000"
+                                  iyy="0.000011" iyz="0.000000"
+                                                 izz="0.000022"/>
+      </inertial>
     </link>
     <!-- joints: main serial chain -->
