Commit message: r2000ib210f: spec limits in degrees.
And use radians(..) to convert.

Easier to compare with the specifications given by Fanuc.

File: fanuc_r2000ib_support/urdf/r2000ib210f_macro.xacro (robot description, xacro)
@@ -115,5 +115,5 @@
       <child link="${prefix}link_1"/>
       <axis xyz="0 0 1"/>
-      <limit lower="-3.14" upper="3.14" effort="0" velocity="1.66"/>
+      <limit lower="${radians(-180)}" upper="${radians(180)}" effort="0" velocity="${radians(95)}"/>
     </joint>
     <joint name="${prefix}joint_2" type="revolute">
@@ -122,5 +122,5 @@
       <child link="${prefix}link_2"/>
       <axis xyz="0 1 0"/>
-      <limit lower="-1.05" upper="1.33" effort="0" velocity="1.57"/>
+      <limit lower="${radians(-60)}" upper="${radians(76)}" effort="0" velocity="${radians(90)}"/>
     </joint>
     <joint name="${prefix}joint_3" type="revolute">
@@ -129,5 +129,5 @@
       <child link="${prefix}link_3"/>
       <axis xyz="0 -1 0"/>
-      <limit lower="-2.3" upper="4.01" effort="0" velocity="1.66"/>
+      <limit lower="${radians(-132)}" upper="${radians(230)}" effort="0" velocity="${radians(95)}"/>
     </joint>
     <joint name="${prefix}joint_4" type="revolute">
@@ -136,5 +136,5 @@
       <child link="${prefix}link_4"/>
       <axis xyz="-1 0 0"/>
-      <limit lower="-6.28" upper="6.28" effort="0" velocity="2.09"/>
+      <limit lower="${radians(-360)}" upper="${radians(360)}" effort="0" velocity="${radians(120)}"/>
     </joint>
     <joint name="${prefix}joint_5" type="revolute">
@@ -143,5 +143,5 @@
       <child link="${prefix}link_5"/>
       <axis xyz="0 -1 0"/>
-      <limit lower="-2.18" upper="2.18" effort="0" velocity="2.09"/>
+      <limit lower="${radians(-125)}" upper="${radians(125)}" effort="0" velocity="${radians(120)}"/>
     </joint>
     <joint name="${prefix}joint_6" type="revolute">
@@ -150,5 +150,5 @@
       <child link="${prefix}link_6"/>
       <axis xyz="0 0 -1"/>
-      <limit lower="-6.28" upper="6.28" effort="0" velocity="3.32"/>
+      <limit lower="${radians(-360)}" upper="${radians(360)}" effort="0" velocity="${radians(190)}"/>
     </joint>
     <!-- ROS-Industrial 'base' frame: base_link to Fanuc World Coordinates transform -->

Commit message: r2000ib210f: spec link lengths with 4 significant digits.

File: fanuc_r2000ib_support/urdf/r2000ib210f_macro.xacro (robot description, xacro)
@@ -111,5 +111,5 @@
     <!-- joints: main serial chain -->
     <joint name="${prefix}joint_1" type="revolute">
-      <origin xyz="0 0 0.67" rpy="0 0 0"/>
+      <origin xyz="0 0 0.670" rpy="0 0 0"/>
       <parent link="${prefix}base_link"/>
       <child link="${prefix}link_1"/>

Commit message: r2000ib210f: translate joints in a single dimension only.
This works better with IKFast and some other tools.

Update link_4 mesh to match.

File: fanuc_r2000ib_support/urdf/r2000ib210f_macro.xacro (robot description, xacro)
@@ -132,5 +132,5 @@
     </joint>
     <joint name="${prefix}joint_4" type="revolute">
-      <origin xyz="1.28 0 0.225" rpy="0 0 0"/>
+      <origin xyz="0 0 0.225" rpy="0 0 0"/>
       <parent link="${prefix}link_3"/>
       <child link="${prefix}link_4"/>
@@ -139,5 +139,5 @@
     </joint>
     <joint name="${prefix}joint_5" type="revolute">
-      <origin xyz="0 0 0" rpy="0 0 0"/>
+      <origin xyz="1.280 0 0" rpy="0 0 0"/>
       <parent link="${prefix}link_4"/>
       <child link="${prefix}link_5"/>

Commit message: r2000ib210f: correct tool0 orientation.
Link-local frames follow REP-103 (chirality). tool0 matches Fanuc's configuration (ie: Z+ forward).

File: fanuc_r2000ib_support/urdf/r2000ib210f_macro.xacro (robot description, xacro)
@@ -146,5 +146,5 @@
     </joint>
     <joint name="${prefix}joint_6" type="revolute">
-      <origin xyz="0.235 0 0" rpy="0 ${pi/2} 0"/>
+      <origin xyz="0.235 0 0" rpy="0 0 0"/>
       <parent link="${prefix}link_5"/>
       <child link="${prefix}link_6"/>
@@ -169,5 +169,5 @@
     <link name="${prefix}tool0" />
     <joint name="${prefix}link_6-tool0" type="fixed">
-      <origin xyz="0 0 0" rpy="0 0 0" />
+      <origin xyz="0 0 0" rpy="${pi} ${-pi/2.0} 0" />
       <parent link="${prefix}flange" />
       <child link="${prefix}tool0" />

Commit message: r2000ib210f: fix joint_6 axis rotation direction.
Joint rotates around X+.

Checked against Fig 3.1 (Basic Specifications - Robot Configuration) of the operator's manual.

File: fanuc_r2000ib_support/urdf/r2000ib210f_macro.xacro (robot description, xacro)
@@ -149,5 +149,5 @@
       <parent link="${prefix}link_5"/>
       <child link="${prefix}link_6"/>
-      <axis xyz="0 0 -1"/>
+      <axis xyz="-1 0 0"/>
       <limit lower="${radians(-360)}" upper="${radians(360)}" effort="0" velocity="${radians(190)}"/>
     </joint>
