Commit message: removed meshes changed package.xml and modified .xacro

File: fanuc_r2000ic_support/urdf/r2000ic210f_macro.xacro (robot description, xacro)
@@ -8,5 +8,5 @@
         <origin xyz="0 0 0" rpy="0 0 0"/>
         <geometry>
-          <mesh filename="package://fanuc_r2000ic_support/meshes/r2000ic210f/visual/base_link.stl"/>
+          <mesh filename="package://fanuc_r2000ic_support/meshes/r2000ic165f/visual/base_link.stl"/>
         </geometry>
         <xacro:material_fanuc_gray40 />
@@ -15,5 +15,5 @@
         <origin xyz="0 0 0" rpy="0 0 0"/>
         <geometry>
-          <mesh filename="package://fanuc_r2000ic_support/meshes/r2000ic210f/collision/base_link.stl"/>
+          <mesh filename="package://fanuc_r2000ic_support/meshes/r2000ic165f/collision/base_link.stl"/>
         </geometry>
       </collision>
@@ -23,5 +23,5 @@
         <origin xyz="0 0 0" rpy="0 0 0"/>
         <geometry>
-          <mesh filename="package://fanuc_r2000ic_support/meshes/r2000ic210f/visual/link_1.stl"/>
+          <mesh filename="package://fanuc_r2000ic_support/meshes/r2000ic165f/visual/link_1.stl"/>
         </geometry>
         <xacro:material_fanuc_yellow />
@@ -30,5 +30,5 @@
         <origin xyz="0 0 0" rpy="0 0 0"/>
         <geometry>
-          <mesh filename="package://fanuc_r2000ic_support/meshes/r2000ic210f/collision/link_1.stl"/>
+          <mesh filename="package://fanuc_r2000ic_support/meshes/r2000ic165f/collision/link_1.stl"/>
         </geometry>
       </collision>
@@ -38,5 +38,5 @@
         <origin xyz="0 0 0" rpy="0 0 0"/>
         <geometry>
-          <mesh filename="package://fanuc_r2000ic_support/meshes/r2000ic210f/visual/link_2.stl"/>
+          <mesh filename="package://fanuc_r2000ic_support/meshes/r2000ic165f/visual/link_2.stl"/>
         </geometry>
         <xacro:material_fanuc_yellow />
@@ -45,5 +45,5 @@
         <origin xyz="0 0 0" rpy="0 0 0"/>
         <geometry>
-          <mesh filename="package://fanuc_r2000ic_support/meshes/r2000ic210f/collision/link_2.stl"/>
+          <mesh filename="package://fanuc_r2000ic_support/meshes/r2000ic165f/collision/link_2.stl"/>
         </geometry>
       </collision>
@@ -53,5 +53,5 @@
         <origin xyz="0 0 0" rpy="0 0 0"/>
         <geometry>
-          <mesh filename="package://fanuc_r2000ic_support/meshes/r2000ic210f/visual/link_3.stl"/>
+          <mesh filename="package://fanuc_r2000ic_support/meshes/r2000ic165f/visual/link_3.stl"/>
         </geometry>
         <xacro:material_fanuc_yellow />
@@ -60,5 +60,5 @@
         <origin xyz="0 0 0" rpy="0 0 0"/>
         <geometry>
-          <mesh filename="package://fanuc_r2000ic_support/meshes/r2000ic210f/collision/link_3.stl"/>
+          <mesh filename="package://fanuc_r2000ic_support/meshes/r2000ic165f/collision/link_3.stl"/>
         </geometry>
       </collision>
@@ -68,5 +68,5 @@
         <origin xyz="0 0 0" rpy="0 0 0"/>
         <geometry>
-          <mesh filename="package://fanuc_r2000ic_support/meshes/r2000ic210f/visual/link_4.stl"/>
+          <mesh filename="package://fanuc_r2000ic_support/meshes/r2000ic165f/visual/link_4.stl"/>
         </geometry>
         <xacro:material_fanuc_yellow />
@@ -75,5 +75,5 @@
         <origin xyz="0 0 0" rpy="0 0 0"/>
         <geometry>
-          <mesh filename="package://fanuc_r2000ic_support/meshes/r2000ic210f/collision/link_4.stl"/>
+          <mesh filename="package://fanuc_r2000ic_support/meshes/r2000ic165f/collision/link_4.stl"/>
         </geometry>
       </collision>
@@ -83,5 +83,5 @@
         <origin xyz="0 0 0" rpy="0 0 0"/>
         <geometry>
-          <mesh filename="package://fanuc_r2000ic_support/meshes/r2000ic210f/visual/link_5.stl"/>
+          <mesh filename="package://fanuc_r2000ic_support/meshes/r2000ic165f/visual/link_5.stl"/>
         </geometry>
         <xacro:material_fanuc_yellow />
@@ -90,5 +90,5 @@
         <origin xyz="0 0 0" rpy="0 0 0"/>
         <geometry>
-          <mesh filename="package://fanuc_r2000ic_support/meshes/r2000ic210f/collision/link_5.stl"/>
+          <mesh filename="package://fanuc_r2000ic_support/meshes/r2000ic165f/collision/link_5.stl"/>
         </geometry>
       </collision>
@@ -98,5 +98,5 @@
         <origin xyz="0 0 0" rpy="0 0 0"/>
         <geometry>
-          <mesh filename="package://fanuc_r2000ic_support/meshes/r2000ic210f/visual/link_6.stl"/>
+          <mesh filename="package://fanuc_r2000ic_support/meshes/r2000ic165f/visual/link_6.stl"/>
         </geometry>
         <xacro:material_fanuc_black />
@@ -105,5 +105,5 @@
         <origin xyz="0 0 0" rpy="0 0 0"/>
         <geometry>
-          <mesh filename="package://fanuc_r2000ic_support/meshes/r2000ic210f/collision/link_6.stl"/>
+          <mesh filename="package://fanuc_r2000ic_support/meshes/r2000ic165f/collision/link_6.stl"/>
         </geometry>
       </collision>
