Commit message: added support for r2000ic-210l

File: fanuc_r2000ic_support/urdf/r2000ic210l_macro.xacro (robot description, xacro)
@@ -1,6 +1,6 @@
-<?xml version="1.0" ?>
+<?xml version="1.0"?>
 <robot xmlns:xacro="http://wiki.ros.org/xacro">
   <xacro:include filename="$(find fanuc_resources)/urdf/common_materials.xacro"/>
-  <xacro:macro name="fanuc_crx10ial" params="prefix">
+  <xacro:macro name="fanuc_r2000ic210l" params="prefix">
     <!-- links: main serial chain -->
     <link name="${prefix}base_link">
@@ -8,12 +8,12 @@
         <origin xyz="0 0 0" rpy="0 0 0"/>
         <geometry>
-          <mesh filename="package://fanuc_crx10ia_support/meshes/crx10ial/visual/base_link.stl"/>
+          <mesh filename="package://fanuc_r2000ic_support/meshes/r2000ic210l/visual/base_link.stl"/>
         </geometry>
-        <xacro:material_fanuc_gray24 />
+        <xacro:material_fanuc_gray40 />
       </visual>
       <collision>
         <origin xyz="0 0 0" rpy="0 0 0"/>
         <geometry>
-          <mesh filename="package://fanuc_crx10ia_support/meshes/crx10ial/collision/base_link.stl"/>
+          <mesh filename="package://fanuc_r2000ic_support/meshes/r2000ic210l/collision/base_link.stl"/>
         </geometry>
       </collision>
@@ -23,12 +23,12 @@
         <origin xyz="0 0 0" rpy="0 0 0"/>
         <geometry>
-          <mesh filename="package://fanuc_crx10ia_support/meshes/crx10ial/visual/link_1.stl"/>
+          <mesh filename="package://fanuc_r2000ic_support/meshes/r2000ic210l/visual/link_1.stl"/>
         </geometry>
-        <xacro:material_fanuc_white />
+        <xacro:material_fanuc_yellow />
       </visual>
       <collision>
         <origin xyz="0 0 0" rpy="0 0 0"/>
         <geometry>
-          <mesh filename="package://fanuc_crx10ia_support/meshes/crx10ial/collision/link_1.stl"/>
+          <mesh filename="package://fanuc_r2000ic_support/meshes/r2000ic210l/collision/link_1.stl"/>
         </geometry>
       </collision>
@@ -38,12 +38,12 @@
         <origin xyz="0 0 0" rpy="0 0 0"/>
         <geometry>
-          <mesh filename="package://fanuc_crx10ia_support/meshes/crx10ial/visual/link_2.stl"/>
+          <mesh filename="package://fanuc_r2000ic_support/meshes/r2000ic210l/visual/link_2.stl"/>
         </geometry>
-        <xacro:material_fanuc_white />
+        <xacro:material_fanuc_yellow />
       </visual>
       <collision>
         <origin xyz="0 0 0" rpy="0 0 0"/>
         <geometry>
-          <mesh filename="package://fanuc_crx10ia_support/meshes/crx10ial/collision/link_2.stl"/>
+          <mesh filename="package://fanuc_r2000ic_support/meshes/r2000ic210l/collision/link_2.stl"/>
         </geometry>
       </collision>
@@ -53,12 +53,12 @@
         <origin xyz="0 0 0" rpy="0 0 0"/>
         <geometry>
-          <mesh filename="package://fanuc_crx10ia_support/meshes/crx10ial/visual/link_3.stl"/>
+          <mesh filename="package://fanuc_r2000ic_support/meshes/r2000ic210l/visual/link_3.stl"/>
         </geometry>
-        <xacro:material_fanuc_white />
+        <xacro:material_fanuc_yellow />
       </visual>
       <collision>
         <origin xyz="0 0 0" rpy="0 0 0"/>
         <geometry>
-          <mesh filename="package://fanuc_crx10ia_support/meshes/crx10ial/collision/link_3.stl"/>
+          <mesh filename="package://fanuc_r2000ic_support/meshes/r2000ic210l/collision/link_3.stl"/>
         </geometry>
       </collision>
@@ -68,12 +68,12 @@
         <origin xyz="0 0 0" rpy="0 0 0"/>
         <geometry>
-          <mesh filename="package://fanuc_crx10ia_support/meshes/crx10ial/visual/link_4.stl"/>
+          <mesh filename="package://fanuc_r2000ic_support/meshes/r2000ic210l/visual/link_4.stl"/>
         </geometry>
-        <xacro:material_fanuc_white />
+        <xacro:material_fanuc_yellow />
       </visual>
       <collision>
         <origin xyz="0 0 0" rpy="0 0 0"/>
         <geometry>
-          <mesh filename="package://fanuc_crx10ia_support/meshes/crx10ial/collision/link_4.stl"/>
+          <mesh filename="package://fanuc_r2000ic_support/meshes/r2000ic210l/collision/link_4.stl"/>
         </geometry>
       </collision>
@@ -83,12 +83,12 @@
         <origin xyz="0 0 0" rpy="0 0 0"/>
         <geometry>
-          <mesh filename="package://fanuc_crx10ia_support/meshes/crx10ial/visual/link_5.stl"/>
+          <mesh filename="package://fanuc_r2000ic_support/meshes/r2000ic210l/visual/link_5.stl"/>
         </geometry>
-        <xacro:material_fanuc_white />
+        <xacro:material_fanuc_yellow />
       </visual>
       <collision>
         <origin xyz="0 0 0" rpy="0 0 0"/>
         <geometry>
-          <mesh filename="package://fanuc_crx10ia_support/meshes/crx10ial/collision/link_5.stl"/>
+          <mesh filename="package://fanuc_r2000ic_support/meshes/r2000ic210l/collision/link_5.stl"/>
         </geometry>
       </collision>
@@ -98,12 +98,12 @@
         <origin xyz="0 0 0" rpy="0 0 0"/>
         <geometry>
-          <mesh filename="package://fanuc_crx10ia_support/meshes/crx10ial/visual/link_6.stl"/>
+          <mesh filename="package://fanuc_r2000ic_support/meshes/r2000ic210l/visual/link_6.stl"/>
         </geometry>
-        <xacro:material_fanuc_gray24 />
+        <xacro:material_fanuc_black />
       </visual>
       <collision>
         <origin xyz="0 0 0" rpy="0 0 0"/>
         <geometry>
-          <mesh filename="package://fanuc_crx10ia_support/meshes/crx10ial/collision/link_6.stl"/>
+          <mesh filename="package://fanuc_r2000ic_support/meshes/r2000ic210l/collision/link_6.stl"/>
         </geometry>
       </collision>
@@ -111,49 +111,49 @@
     <!-- joints: main serial chain -->
     <joint name="${prefix}joint_1" type="revolute">
-      <origin xyz="0 0 0.245" rpy="0 0 0" />
-      <parent link="${prefix}base_link" />
-      <child link="${prefix}link_1" />
-      <axis xyz="0 0 1" />
-      <limit effort="0" lower="-3.14159" upper="3.14159" velocity="2.0944" />
+      <origin xyz="0 0 0.67" rpy="0 0 0"/>
+      <parent link="${prefix}base_link"/>
+      <child link="${prefix}link_1"/>
+      <axis xyz="0 0 1"/>
+      <limit lower="${radians(-185)}" upper="${radians(185)}" effort="0" velocity="${radians(105)}"/>
     </joint>
     <joint name="${prefix}joint_2" type="revolute">
-      <origin xyz="0 0 0" rpy="0 0 0" />
-      <parent link="${prefix}link_1" />
-      <child link="${prefix}link_2" />
-      <axis xyz="0 1 0" />
-      <limit effort="0" lower="-3.14159" upper="3.14159" velocity="2.0944" />
+      <origin xyz="0.312 0 0" rpy="0 0 0"/>
+      <parent link="${prefix}link_1"/>
+      <child link="${prefix}link_2"/>
+      <axis xyz="0 1 0"/>
+      <limit lower="${radians(-60)}" upper="${radians(76)}" effort="0" velocity="${radians(90)}"/>
     </joint>
     <joint name="${prefix}joint_3" type="revolute">
-      <origin xyz="0 0 0.710" rpy="0 0 0" />
-      <parent link="${prefix}link_2" />
-      <child link="${prefix}link_3" />
-      <axis xyz="0 -1 0" />
-      <limit effort="0" lower="-4.71239" upper="4.71239" velocity="3.14159" />
+      <origin xyz="0 0 1.075" rpy="0 0 0"/>
+      <parent link="${prefix}link_2"/>
+      <child link="${prefix}link_3"/>
+      <axis xyz="0 -1 0"/>
+      <limit lower="${radians(-121)}" upper="${radians(180)}" effort="0" velocity="${radians(85)}"/>
     </joint>
     <joint name="${prefix}joint_4" type="revolute">
-      <origin xyz="0 0 0" rpy="0 0 0"/>
+      <origin xyz="0 0 0.225" rpy="0 0 0"/>
       <parent link="${prefix}link_3"/>
       <child link="${prefix}link_4"/>
       <axis xyz="-1 0 0"/>
-      <limit effort="0" lower="-3.31613" upper="3.31613" velocity="3.14159" />
+      <limit lower="${radians(-360)}" upper="${radians(360)}" effort="0" velocity="${radians(120)}"/>
     </joint>
     <joint name="${prefix}joint_5" type="revolute">
-      <origin xyz="0.540 -0.150 0" rpy="0 0 0"/>
+      <origin xyz="1.730 0 0" rpy="0 0 0"/>
       <parent link="${prefix}link_4"/>
       <child link="${prefix}link_5"/>
       <axis xyz="0 -1 0"/>
-      <limit effort="0" lower="-3.14159" upper="3.14159" velocity="3.14159" />
+      <limit lower="${radians(-125)}" upper="${radians(125)}" effort="0" velocity="${radians(120)}"/>
     </joint>
     <joint name="${prefix}joint_6" type="revolute">
-      <origin xyz="0.160 0 0" rpy="0 0 0"/>
+      <origin xyz="0.24 0 0" rpy="0 0 0"/>
       <parent link="${prefix}link_5"/>
       <child link="${prefix}link_6"/>
       <axis xyz="-1 0 0"/>
-      <limit effort="0" lower="-3.31613" upper="3.31613" velocity="3.14159" />
+      <limit lower="${radians(-360)}" upper="${radians(360)}" effort="0" velocity="${radians(200)}"/>
     </joint>
     <!-- ROS-Industrial 'base' frame: base_link to Fanuc World Coordinates transform -->
     <link name="${prefix}base" />
     <joint name="${prefix}base_link-base" type="fixed">
-      <origin xyz="0 0 0.245" rpy="0 0 0"/>
+      <origin xyz="0 0 0.670" rpy="0 0 0"/>
       <parent link="${prefix}base_link"/>
       <child link="${prefix}base"/>
@@ -170,5 +170,5 @@
     <joint name="${prefix}link_6-tool0" type="fixed">
       <origin xyz="0 0 0" rpy="${pi} ${-pi/2.0} 0" />
-      <parent link="${prefix}flange" />
+      <parent link="${prefix}link_6" />
       <child link="${prefix}tool0" />
     </joint>
